File: circets/ActivationModule/Activation_Module/Activation_Module.sch (KiCad schematic (older format))
At the start: 27 parts, among them J1 Service Connector, J2 ctrl line input, J3 Signal_Out, SW1 SW_DIP_x08, SW2 RW, U1 SN54LS08, U2 74HC86, U3 74HC86, U4 74LS32, U5 4078

Commit message: Started Rework on AM
Parts:
- removed J1: Service Connector, symbol Connector:Conn_01x04_Male
- removed J2: ctrl line input, symbol Connector:Conn_01x08_Male
- removed J3: Signal_Out, symbol Connector:Conn_01x02_Female
- removed R10, R11, R12, R13, R14, R15, R16, R9, R?: 10k, symbol Device:R
- removed SW1: SW_DIP_x08, symbol Switch:SW_DIP_x08
- removed SW2: RW, symbol Switch:SW_DIP_x01
- removed U1: SN54LS08, symbol Computer_Component_Library:SN54LS08
- removed U2, U3: 74HC86, symbol 74xx:74HC86
- removed U4: 74LS32, symbol 74xx:74LS32
- removed U5: 4078, symbol 4xxx_IEEE:4078
- added SW? (x2): SW_DIP_x04, symbol Switch:SW_DIP_x04
- added U1, U2, U3, U4: 74LS86, symbol 74xx:74LS86
- added U5, U6, U7, U8: 74LS32, symbol 74xx:74LS32
Connections:
- net labels removed: CLK_F, CLK_R, GND, Signal_Out_1, Signal_Out_2, Vcc
- wire segments 211 -> 134

Commit message: Revised Activation Module
Parts:
- added Enable_Connector: Conn_01x03_Female, symbol Connector:Conn_01x03_Female
- added J1, J4: Bus_Connector, symbol Computer_Component_Library:Bus_Connector
- added J2: To_Bus, symbol Connector:Conn_01x16_Female
- added J3: From_Bus, symbol Connector:Conn_01x16_Female
- added J5: Mode_R, symbol Connector:Conn_01x03_Female
- added J6: Mode_W, symbol Connector:Conn_01x03_Female
- added U11, U12, U? (x10): 74HC541, symbol Computer_Component_Library:74HC541
- added U9: 74HC00, symbol 74xx:74HC00
Connections:
- net at U1.2: now also J1.40 (WE1:3)
- net at U1.5: now also J1.41 (WE1:4)
- net at U1.10: now also J1.42 (WE1:5)
- net at U1.13: now also J1.43 (WE1:6)
- net +5V: now reaches U1.14 (VCC)
- net +5V: now also SW?.1, SW?.1, SW?.2, SW?.2, SW?.3, SW?.3, SW?.4, SW?.4, U2.14 (VCC), U3.14 (VCC), U4.7 (GND), U5.14 (VCC), U6.14 (VCC), U7.14 (VCC), U8.14 (VCC), J4.2 (Vcc), U11.20 (Vcc), U12.20 (Vcc), U9.14 (VCC), U?.20 (Vcc), U?.20 (Vcc), U?.20 (Vcc), U?.20 (Vcc), U?.20 (Vcc), U?.20 (Vcc), U?.20 (Vcc), U?.20 (Vcc), U?.20 (Vcc), U?.20 (Vcc)
- net GND: now reaches U1.7 (GND)
- net GND: now also R1.1, R2.1, R3.1, R4.1, R5.1, R6.1, R7.1, R8.1, U2.7 (GND), U3.7 (GND), U4.14 (VCC), U5.7 (GND), U6.7 (GND), U7.7 (GND), U8.7 (GND), J4.1 (GND), U11.1 (~G1), U11.10 (GND), U12.1 (~G1), U12.10 (GND), U9.7 (GND), U?.1 (~G1), U?.1 (~G1), U?.10 (GND), U?.10 (GND), U?.10 (GND), U?.10 (GND), U?.10 (GND), U?.10 (GND), U?.10 (GND), U?.10 (GND), U?.10 (GND), U?.10 (GND), U?.19 (~G2), U?.19 (~G2), U?.19 (~G2), U?.19 (~G2)
- net at U2.2: now also J1.61 (RE2:3)
- net at U2.5: now also J1.62 (RE2:4)
- net at U2.10: now also J1.63 (RE2:5)
- net at U2.13: now also J1.64 (RE2:6)
- net at U3.2: now also J1.54 (RE1:3)
- net at U3.5: now also J1.55 (RE1:4)
- net at U3.10: now also J1.56 (RE1:5)
- net at U3.13: now also J1.57 (RE1:6)
- net at U4.2: now also J1.47 (WE2:3)
- net at U4.5: now also J1.48 (WE2:4)
- net at U4.10: now also J1.49 (WE2:5)
- net at U4.13: now also J1.50 (WE2:6)
- net at U5.12, U5.8: now also U?.1 (~G1), U?.1 (~G1), U?.1 (~G1)
- net RE: now reaches U5.11
- net RE: now also Enable_Connector.3 (Pin_3)
- net at U5.13, U6.8: now also U?.1 (~G1), U?.1 (~G1), U?.1 (~G1)
- net at U7.8, U8.13: now also U?.1 (~G1), U?.19 (~G2), U?.19 (~G2)
- net at U8.12, U8.8: now also U11.19 (~G2), U12.19 (~G2), U?.1 (~G1)
- net at U8.11: now also U9.1, U9.9
- new net: J4.4 (CLK_F), U9.2
- new net: U9.3, U9.4, U9.5
- new net: J4.3 (CLK_R), U9.10
- new net: U9.12, U9.13, U9.8
- new net: J3.16 (Pin_16), U11.11 (Y8), U?.11 (Y8)
- new net: J3.15 (Pin_15), U11.12 (Y7), U?.12 (Y7)
- new net: J3.14 (Pin_14), U11.13 (Y6), U?.13 (Y6)
- new net: J3.13 (Pin_13), U11.14 (Y5), U?.14 (Y5)
- new net: J3.12 (Pin_12), U11.15 (Y4), U?.15 (Y4)
- new net: J3.11 (Pin_11), U11.16 (Y3), U?.16 (Y3)
- new net: J3.10 (Pin_10), U11.17 (Y2), U?.17 (Y2)
- new net: J3.9 (Pin_9), U11.18 (Y1), U?.18 (Y1)
- new net: J1.13 (BUS1:8), U11.2 (A1), U?.11 (Y8)
- new net: J1.14 (BUS1:9), U11.3 (A2), U?.12 (Y7)
- new net: J1.15 (BUS1:A), U11.4 (A3), U?.13 (Y6)
- new net: J1.16 (BUS1:B), U11.5 (A4), U?.14 (Y5)
- new net: J1.17 (BUS1:C), U11.6 (A5), U?.15 (Y4)
- new net: J1.18 (BUS1:D), U11.7 (A6), U?.16 (Y3)
- new net: J1.19 (BUS1:E), U11.8 (A7), U?.17 (Y2)
- new net: J1.20 (BUS1:F), U11.9 (A8), U?.18 (Y1)
- new net: J3.8 (Pin_8), U12.11 (Y8), U?.11 (Y8)
- new net: J3.7 (Pin_7), U12.12 (Y7), U?.12 (Y7)
- new net: J3.6 (Pin_6), U12.13 (Y6), U?.13 (Y6)
- new net: J3.5 (Pin_5), U12.14 (Y5), U?.14 (Y5)
- new net: J3.4 (Pin_4), U12.15 (Y4), U?.15 (Y4)
- new net: J3.3 (Pin_3), U12.16 (Y3), U?.16 (Y3)
- new net: J3.2 (Pin_2), U12.17 (Y2), U?.17 (Y2)
- new net: J3.1 (Pin_1), U12.18 (Y1), U?.18 (Y1)
- new net: J1.5 (BUS1:0), U12.2 (A1), U?.18 (Y1)
- new net: J1.6 (BUS1:1), U12.3 (A2), U?.17 (Y2)
- new net: J1.7 (BUS1:2), U12.4 (A3), U?.16 (Y3)
- new net: J1.8 (BUS1:3), U12.5 (A4), U?.15 (Y4)
- new net: J1.9 (BUS1:4), U12.6 (A5), U?.14 (Y5)
- new net: J1.10 (BUS1:5), U12.7 (A6), U?.13 (Y6)
- new net: J1.11 (BUS1:6), U12.8 (A7), U?.12 (Y7)
- new net: J1.12 (BUS1:7), U12.9 (A8), U?.11 (Y8)
- new net: J2.1 (Pin_1), U?.2 (A1), U?.2 (A1)
- new net: J2.10 (Pin_10), U?.3 (A2), U?.3 (A2)
- new net: J2.11 (Pin_11), U?.4 (A3), U?.4 (A3)
- new net: J2.12 (Pin_12), U?.5 (A4), U?.5 (A4)
- new net: J2.13 (Pin_13), U?.6 (A5), U?.6 (A5)
- new net: J2.14 (Pin_14), U?.7 (A6), U?.7 (A6)
- new net: J2.15 (Pin_15), U?.8 (A7), U?.8 (A7)
- new net: J2.16 (Pin_16), U?.9 (A8), U?.9 (A8)
- new net: J2.2 (Pin_2), U?.3 (A2), U?.3 (A2)
- new net: J2.3 (Pin_3), U?.4 (A3), U?.4 (A3)
- new net: J2.4 (Pin_4), U?.5 (A4), U?.5 (A4)
- new net: J2.5 (Pin_5), U?.6 (A5), U?.6 (A5)
- new net: J2.6 (Pin_6), U?.7 (A6), U?.7 (A6)
- new net: J2.7 (Pin_7), U?.8 (A7), U?.8 (A7)
- new net: J2.8 (Pin_8), U?.9 (A8), U?.9 (A8)
- new net: J2.9 (Pin_9), U?.2 (A1), U?.2 (A1)
- new net: J1.21 (BUS2:0), U?.18 (Y1), U?.2 (A1)
- new net: J1.22 (BUS2:1), U?.17 (Y2), U?.3 (A2)
- new net: J1.23 (BUS2:2), U?.16 (Y3), U?.4 (A3)
- new net: J1.24 (BUS2:3), U?.15 (Y4), U?.5 (A4)
- new net: J1.25 (BUS2:4), U?.14 (Y5), U?.6 (A5)
- new net: J1.26 (BUS2:5), U?.13 (Y6), U?.7 (A6)
- new net: J1.27 (BUS2:6), U?.12 (Y7), U?.8 (A7)
- new net: J1.28 (BUS2:7), U?.11 (Y8), U?.9 (A8)
- new net: J1.29 (BUS2:8), U?.11 (Y8), U?.2 (A1)
- new net: J1.30 (BUS2:9), U?.12 (Y7), U?.3 (A2)
- new net: J1.31 (BUS2:A), U?.13 (Y6), U?.4 (A3)
- new net: J1.32 (BUS2:B), U?.14 (Y5), U?.5 (A4)
- new net: J1.33 (BUS2:C), U?.15 (Y4), U?.6 (A5)
- new net: J1.34 (BUS2:D), U?.16 (Y3), U?.7 (A6)
- new net: J1.35 (BUS2:E), U?.17 (Y2), U?.8 (A7)
- new net: J1.36 (BUS2:F), U?.18 (Y1), U?.9 (A8)
- new net: J1.37 (WE1:0), U?.2 (A1)
- new net: J1.38 (WE1:1), U?.3 (A2)
- new net: J1.39 (WE1:2), U?.4 (A3)
- new net: J1.58 (RE2:0), U?.2 (A1)
- new net: J1.59 (RE2:1), U?.3 (A2)
- new net: J1.60 (RE2:2), U?.4 (A3)
- new net: J1.51 (RE1:0), U?.2 (A1)
- new net: J1.52 (RE1:1), U?.3 (A2)
- new net: J1.53 (RE1:2), U?.4 (A3)
- new net: J1.44 (WE2:0), U?.2 (A1)
- new net: J1.45 (WE2:1), U?.3 (A2)
- new net: J1.46 (WE2:2), U?.4 (A3)
- new net: J5.3 (Pin_3), U?.16 (Y3), U?.16 (Y3)
- new net: J5.2 (Pin_2), U?.17 (Y2), U?.17 (Y2)
- new net: J5.1 (Pin_1), U?.18 (Y1), U?.18 (Y1)
- new net: J6.3 (Pin_3), U?.16 (Y3), U?.16 (Y3)
- new net: J6.2 (Pin_2), U?.17 (Y2), U?.17 (Y2)
- new net: J6.1 (Pin_1), U?.18 (Y1), U?.18 (Y1)
- new net WE_F: Enable_Connector.1 (Pin_1), U9.6
- new net WE_R: Enable_Connector.2 (Pin_2), U9.11
Other:
- note added: "Data-Routing"
- note added: "Mode-Router"
- note added: "Read-Enable-Dection"
- note added: "Write-Enable-Detection"
- moved on the sheet: R1, R2, R3, R4, R5, R6, R7, R8, SW?, U1A, U1B, U1C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

Commit message: Fixed Small Issues after build Protype
Parts:
- removed U? (x4): 74HC541, symbol Computer_Component_Library:74HC541
- added U18: 74HC00, symbol 74xx:74HC00
- added U? (x2): 74157, symbol 74xx_IEEE:74157
- R1, R2, R3, R4, R5, R6, R7, R8: value 10k -> 1k
- gave numbers to parts that had none: 6
- renumbered U11 to U13
Connections:
- net +5V: now also U18.7 (GND), U?.16 (VCC), U?.16 (VCC)
- net GND: now also U18.14 (VCC), U?.15 (~EN), U?.15 (~EN), U?.8 (GND), U?.8 (GND)
- net at U2.8: now also U7.4; no longer U7.5
- net at U2.11: now also U7.5; no longer U7.10
- net at U4.8: now also U6.4; no longer U6.5
- net at U4.11: now also U6.5; no longer U6.10
- net at U9.1, U9.9: now also U18.3; no longer U8.11
- net at U10.1 (~G1), U11.1 (~G1), U5.12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: now also U?.1 (A/B)
- net at U6.3: now also U6.9; no longer U6.4
- net at U6.6: now also U6.10; no longer U6.9
- net at U7.3: now also U7.9; no longer U7.4
- net at U7.6: now also U7.10; no longer U7.9
- net at U12.19 (~G2), U13.19 (~G2), U8.12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: now also U?.1 (A/B)
- net at J1.37 (WE1:0): now also U?.2 (I0a)
- net at J1.38 (WE1:1): now also U?.5 (I0b)
- net at J1.39 (WE1:2): now also U?.14 (I0c)
- net at J1.58 (RE2:0): now also U?.2 (I0a)
- net at J1.59 (RE2:1): now also U?.5 (I0b)
- net at J1.60 (RE2:2): now also U?.14 (I0c)
- net at J1.51 (RE1:0): now also U?.3 (I1a)
- net at J1.52 (RE1:1): now also U?.6 (I1b)
- net at J1.53 (RE1:2): now also U?.13 (I1c)
- net at J1.44 (WE2:0): now also U?.3 (I1a)
- net at J1.45 (WE2:1): now also U?.6 (I1b)
- net at J1.46 (WE2:2): now also U?.13 (I1c)
- net at J5.3 (Pin_3): now also U?.12 (Qc)
- net at J5.2 (Pin_2): now also U?.7 (Qb)
- net at J5.1 (Pin_1): now also U?.4 (Qa)
- net at J6.3 (Pin_3): now also U?.12 (Qc)
- net at J6.2 (Pin_2): now also U?.7 (Qb)
- net at J6.1 (Pin_1): now also U?.4 (Qa)
- new net: U18.1, U18.2, U8.11
Other:
- moved on the sheet: Enable_Connector, J4A, J5, J6, U1E, U2E, U3E, U4E, U5E, U6B, U6C, U6D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

Commit message: Made Footprint for 74HC541 and started Footprint for Bus Connector
Parts:
- gave numbers to parts that had none: 4
- renumbered Enable_Connector to Enable_Connector1, J4 to J1, J5 to J4, J6 to J5, U10 to U1, U14 to U10, U9 to U11, U18 to U11, U15 to U12, U16 to U13, U17 to U14, U1 to U15, U3 to U15, U2 to U16, U4 to U16, U5 to U17, U6 to U17, U5 to U18, U6 to U18, U11 to U2, U1 to U3, U4 to U3, U2 to U4, U3 to U4, U7 to U5, U8 to U5, U7 to U6, U8 to U6, U12 to U7, U13 to U8, U18 to U9

Commit message: Transfored Repo to new computer, alot has apperntly chande, let's commit it all!
Parts:
- added C1, C2, C3, C4, C5, C6: 0.1µF, Capacitor_THT:C_Disc_D6.0mm_W2.5mm_P5.00mm, symbol Device:C
- added D1, D2, D3, D4: LED, LED_THT:LED_D4.0mm, symbol Device:LED
- added R10, R11, R12, R9: 220, Resistor_THT:R_Axial_DIN0207_L6.3mm_D2.5mm_P2.54mm_Vertical, symbol Device:R
- J1: footprint (none) -> Computer_Component_Library:BusConnector
- J2, J3: footprint (none) -> Connector_PinHeader_2.54mm:PinHeader_1x16_P2.54mm_Vertical
- J4, J5: footprint (none) -> Connector_PinSocket_2.54mm:PinSocket_1x03_P2.54mm_Vertical
- J6: renamed from Enable_Connector1; value Conn_01x03_Female -> Enable Connector; footprint (none) -> Connector_PinSocket_2.54mm:PinSocket_1x03_P2.54mm_Vertical
- R1, R2, R3, R4, R5, R6, R7, R8: footprint (none) -> Resistor_THT:R_Axial_DIN0207_L6.3mm_D2.5mm_P2.54mm_Vertical
- SW1, SW2: footprint (none) -> Button_Switch_THT:SW_DIP_SPSTx04_Slide_9.78x12.34mm_W7.62mm_P2.54mm
- U1, U10, U12, U13, U14, U2, U7, U8: footprint (none) -> Computer_Component_Library:74HC541-PDIP
- U11, U15, U16, U17, U18, U3, U4, U5, U6, U9: footprint (none) -> Package_DIP:DIP-14_W7.62mm_Socket
- U19, U20: footprint (none) -> Package_DIP:DIP-16_W7.62mm_Socket
Connections:
- net +5V: now also C1.1, C2.1, C3.1, C4.2, C5.2, C6.2, R10.1, R11.1, R12.1, R9.1
- net GND: now also C1.2, C2.2, C3.2, C4.1, C5.1, C6.1
- net RE: now also U18.11; no longer U17.11
- net at U3.8: now also U5.5; no longer U6.5
- net at U3.11: now also U5.10; no longer U6.10
- net at U4.8: now also U6.4; no longer U5.4
- net at U4.11: now also U6.5; no longer U5.5
- net at U15.3: now also U18.1; no longer U17.1
- net at U15.6: now also U18.2; no longer U17.2
- net at U16.3: now also U17.1; no longer U18.1
- net at U16.6: now also U17.2; no longer U18.2
- net at U11.2: now also U11.1, U5.11; no longer J1.4 (CLK_F)
- net at U9.4, U9.5: now also U9.3; no longer U11.3
- net at U17.3: now also U17.9; no longer U18.4
- net at U1.1 (~G1), U18.8, U19.1 (A/B)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: now also U18.12, D3.1 (K); no longer U17.12
- net at U10.1 (~G1), U12.1 (~G1), U17.8: now also U18.13, D4.1 (K); no longer U17.13
- net at U18.3: now also U18.4; no longer U17.9
- net at U6.3: now also U6.9; no longer U5.9
- net at U5.6: now also U5.9; no longer U5.10
- net at U13.19 (~G2), U14.19 (~G2), U5.13: now also U6.8, D2.1 (K); no longer U5.8
- net at U5.3: now also U5.4; no longer U6.4
- net at U6.6: now also U6.10; no longer U6.9
- net at U20.1 (A/B), U5.12, U7.19 (~G2)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: now also U5.8, D1.1 (K); no longer U6.8
- net at J1.13 (BUS1:8), U8.2 (A1): now also U2.18 (Y1); no longer U2.11 (Y8)
- net at J1.14 (BUS1:9), U8.3 (A2): now also U2.17 (Y2); no longer U2.12 (Y7)
- net at J1.15 (BUS1:A), U8.4 (A3): now also U2.16 (Y3); no longer U2.13 (Y6)
- net at J1.16 (BUS1:B), U8.5 (A4): now also U2.15 (Y4); no longer U2.14 (Y5)
- net at J1.17 (BUS1:C), U8.6 (A5): now also U2.14 (Y5); no longer U2.15 (Y4)
- net at J1.18 (BUS1:D), U8.7 (A6): now also U2.13 (Y6); no longer U2.16 (Y3)
- net at J1.19 (BUS1:E), U8.8 (A7): now also U2.12 (Y7); no longer U2.17 (Y2)
- net at J1.20 (BUS1:F), U8.9 (A8): now also U2.11 (Y8); no longer U2.18 (Y1)
- net at J1.29 (BUS2:8), U14.2 (A1): no longer U12.11 (Y8)
- net at J1.30 (BUS2:9), U14.3 (A2): now also U12.17 (Y2); no longer U12.12 (Y7)
- net at J1.31 (BUS2:A), U14.4 (A3): now also U12.16 (Y3); no longer U12.13 (Y6)
- net at J1.32 (BUS2:B), U14.5 (A4): now also U12.15 (Y4); no longer U12.14 (Y5)
- net at J1.33 (BUS2:C), U14.6 (A5): now also U12.14 (Y5); no longer U12.15 (Y4)
- net at J1.34 (BUS2:D), U14.7 (A6): now also U12.13 (Y6); no longer U12.16 (Y3)
- net at J1.35 (BUS2:E), U14.8 (A7): now also U12.12 (Y7); no longer U12.17 (Y2)
- net at J1.36 (BUS2:F), U14.9 (A8): now also U12.11 (Y8); no longer U12.18 (Y1)
- new net: U11.3, U9.1, U9.9
- new net: J1.4 (CLK_F), U9.2
- new net: D1.2 (A), R9.2
- new net: D2.2 (A), R10.2
- new net: D3.2 (A), R11.2
- new net: D4.2 (A), R12.2
Other:
- moved on the sheet: U11A, U11B, U11C, U11D, U17A, U17D, U18A, U18D, U5B, U5C, U6B, U6C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
