File: circets/register_file/register_file_kicad/register_file_kicad.sch (KiCad schematic (older format))
At the start: 60 parts, among them J0 D_In, J1 A_Out, J2 B_Out, J3 D_Sel, J4 A_Sel, J5 B_Sel, J6 Service_Connector, J7 Controll_Connector, U1 74HC573, U10 74HC573, U11 74HC573, U12 74HC573, U13 74HC573, U14 74HC573, U15 74HC573, U16 74HC573, U17 74HC00, U18 74LS139, U19 74LS139, U2 74HC573, U20 74LS139, U3 74HC573, U4 74HC573, U5 74HC573, U6 74HC573, U7 74HC573, U8 74HC573, U9 74HC573

Commit message: Transfored Repo to new computer, alot has apperntly chande, let's commit it all!
Parts:
- removed J0: D_In, symbol Connector:Conn_01x16_Female
- removed J1: A_Out, symbol Connector:Conn_01x16_Female
- removed J2: B_Out, symbol Connector:Conn_01x16_Female
- removed J3: D_Sel, symbol Connector:Conn_01x03_Female
- removed J4: A_Sel, symbol Connector:Conn_01x03_Female
- removed J5: B_Sel, symbol Connector:Conn_01x03_Female
- removed J6: Service_Connector, symbol Connector:Conn_01x04_Female
- removed J7: Controll_Connector, symbol Connector:Conn_01x04_Female
- removed U1, U10, U11, U12, U13, U14, U15, U16, U2, U3, U4, U5, U6, U7, U8, U9: 74HC573, symbol Computer_Component_Library:74HC573
- removed U17: 74HC00, symbol 74xx:74HC00
- removed U18, U19, U20: 74LS139, symbol 74xx:74LS139
- removed U? (x32): 74HC541, symbol Computer_Component_Library:74HC541
- added J?: D_In, symbol Connector:Conn_01x16_Female
- added J?: A_Out, symbol Connector:Conn_01x16_Female
- added J?: B_Out, symbol Connector:Conn_01x16_Female
- added U? (x10): 74HC573, symbol Computer_Component_Library:74HC573
- added U? (x16): 74HC541, symbol Computer_Component_Library:74HC541
Connections:
- net labels removed: A_Out_1, A_Out_10, A_Out_11, A_Out_12, A_Out_13, A_Out_14, A_Out_15, A_Out_16, A_Out_2, A_Out_3, A_Out_4, A_Out_5, A_Out_6, A_Out_7, A_Out_8, A_Out_9, B_Out_1, B_Out_10, B_Out_11, B_Out_12, B_Out_13, B_Out_14, B_Out_15, B_Out_16, B_Out_2, B_Out_3, B_Out_4, B_Out_5, B_Out_6, B_Out_7, B_Out_8, B_Out_9, CLK_F, CLK_R, D_In_1, D_In_10, D_In_11, D_In_12, D_In_13, D_In_14, D_In_15, D_In_16, D_In_2, D_In_3, D_In_4, D_In_5, D_In_6, D_In_7, D_In_8, D_In_9, D_Out_A_1, D_Out_A_10, D_Out_A_11, D_Out_A_12, D_Out_A_13, D_Out_A_14, D_Out_A_15, D_Out_A_16, D_Out_A_2, D_Out_A_3, D_Out_A_4, D_Out_A_5, D_Out_A_6, D_Out_A_7, D_Out_A_8, D_Out_A_9, D_Out_B_1, D_Out_B_10, D_Out_B_11, D_Out_B_12, D_Out_B_13, D_Out_B_14, D_Out_B_15, D_Out_B_16, D_Out_B_2, D_Out_B_3, D_Out_B_4, D_Out_B_5, D_Out_B_6, D_Out_B_7, D_Out_B_8, D_Out_B_9, D_Out_C_1, D_Out_C_10, D_Out_C_11, D_Out_C_12, D_Out_C_13, D_Out_C_14, D_Out_C_15, D_Out_C_16, D_Out_C_2, D_Out_C_3, D_Out_C_4, D_Out_C_5, D_Out_C_6, D_Out_C_7, D_Out_C_8, D_Out_C_9, D_Out_D_1, D_Out_D_10, D_Out_D_11, D_Out_D_12, D_Out_D_13, D_Out_D_14, D_Out_D_15, D_Out_D_16, D_Out_D_2, D_Out_D_3, D_Out_D_4, D_Out_D_5, D_Out_D_6, D_Out_D_7, D_Out_D_8, D_Out_D_9, D_Out_F_1, D_Out_F_10, D_Out_F_11, D_Out_F_12, D_Out_F_13, D_Out_F_14, D_Out_F_15, D_Out_F_16, D_Out_F_2, D_Out_F_3, D_Out_F_4, D_Out_F_5, D_Out_F_6, D_Out_F_7, D_Out_F_8, D_Out_F_9, D_Out_IP_1, D_Out_IP_10, D_Out_IP_11, D_Out_IP_12, D_Out_IP_13, D_Out_IP_14, D_Out_IP_15, D_Out_IP_16, D_Out_IP_2, D_Out_IP_3, D_Out_IP_4, D_Out_IP_5, D_Out_IP_6, D_Out_IP_7, D_Out_IP_8, D_Out_IP_9, D_Out_SP_1, D_Out_SP_10, D_Out_SP_11, D_Out_SP_12, D_Out_SP_13, D_Out_SP_14, D_Out_SP_15, D_Out_SP_16, D_Out_SP_2, D_Out_SP_3, D_Out_SP_4, D_Out_SP_5, D_Out_SP_6, D_Out_SP_7, D_Out_SP_8, D_Out_SP_9, R_Sup, S_SUP, Vcc, WE, ZERO_ONE
- wire segments 1389 -> 1070
Other:
- note removed: "A"
- note removed: "B"
- note removed: "C"
- note removed: "D"
- note removed: "FLAG"
- note removed: "IP\n"
- note removed: "SP\n"
- note removed: "ZERO\n"

Commit message: Reworked Register Logic-Schematic and Kicad-Schematic
Parts:
- removed U? (x2): 74HC573, symbol Computer_Component_Library:74HC573
- added J?: Const_In, symbol Connector:Conn_01x16_Female
- added J?: Conn_01x05_Female, symbol Connector:Conn_01x05_Female
- added J?: Flag_Out, symbol Connector:Conn_01x16_Female
- added J?: Conn_01x16_Female, symbol Connector:Conn_01x16_Female
- added J?: D_Sel, symbol Connector:Conn_01x03_Female
- added J?: A_Sel, symbol Connector:Conn_01x03_Female
- added J?: B_Sel, symbol Connector:Conn_01x03_Female
- added J?: Bus_Connector, symbol Computer_Component_Library:Bus_Connector
- added U? (x8): 74HC573, symbol register_file_kicad-rescue:74HC573-Computer_Component_Library
- added U? (x16): 74HC541, symbol register_file_kicad-rescue:74HC541-Computer_Component_Library
- added U? (x3): 74HC00, symbol 74xx:74HC00
- added U? (x2): 4027, symbol 4xxx:4027
- added U? (x15): 74LS08, symbol 74xx:74LS08
- added U? (x3): 74HC137, symbol 74xx:74HC137
- added U?: 74HC540, symbol Computer_Component_Library:74HC540
- added U? (x2): 74HC541, symbol Computer_Component_Library:74HC541
- U? (x8): symbol Computer_Component_Library:74HC573 -> register_file_kicad-rescue:74HC573-Computer_Component_Library
- U? (x16): symbol Computer_Component_Library:74HC541 -> register_file_kicad-rescue:74HC541-Computer_Component_Library
Connections:
- net GND: now also U?.10 (GND), U?.10 (GND), U?.10 (GND), U?.10 (GND), U?.10 (GND), U?.10 (GND), J?.1 (GND), U?.10 (GND), U?.10 (GND), U?.10 (GND), U?.10 (GND), U?.10 (GND), U?.10 (GND), U?.10 (GND), U?.10 (GND), U?.10 (GND), U?.10 (GND), U?.10 (GND), U?.10 (GND), U?.10 (GND), U?.10 (GND), U?.10 (GND), U?.10 (GND), U?.10 (GND), U?.10 (GND), U?.10 (GND), U?.10 (GND), U?.10 (GND), U?.10 (GND), U?.10 (GND), U?.10 (GND), U?.10 (GND), U?.10 (GND), U?.10 (GND), U?.4 (~LE), U?.4 (~LE), U?.4 (~LE), U?.5 (~E1), U?.5 (~E1), U?.7 (GND), U?.7 (GND), U?.7 (GND), U?.7 (GND), U?.8 (GND), U?.8 (GND), U?.8 (GND), U?.8 (VSS)
- net at U?.9 (A8), U?.9 (A8): now also U?.2 (A1), U?.2 (A1), U?.3 (A2), U?.3 (A2), U?.3 (A2), U?.3 (A2), U?.4 (A3), U?.4 (A3), U?.4 (A3), U?.4 (A3), U?.5 (A4), U?.5 (A4), U?.5 (A4), U?.5 (A4), U?.6 (A5), U?.6 (A5), U?.6 (A5), U?.6 (A5), U?.7 (A6), U?.7 (A6), U?.7 (A6), U?.7 (A6), U?.8 (A7), U?.8 (A7), U?.8 (A7), U?.8 (A7), U?.9 (A8), U?.9 (A8)
- net Zero_One: now reaches U?.2 (A1), U?.2 (A1)
- net Zero_One: now also J?.4 (Pin_4)
- net at U?.19 (1Q), U?.2 (1D), U?.2 (1D)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: now also U?.2 (1D), U?.2 (1D), U?.2 (1D), U?.2 (1D) (x2)
- net +5V: now reaches U?.20 (VCC), U?.20 (VCC), U?.20 (VCC), U?.20 (VCC), U?.20 (VCC), U?.20 (VCC)
- net +5V: now also U?.20 (VCC), U?.20 (VCC), U?.20 (Vcc), U?.20 (Vcc), U?.20 (Vcc), U?.20 (Vcc), U?.20 (Vcc), U?.20 (Vcc), U?.20 (Vcc), U?.20 (Vcc), U?.20 (Vcc), U?.20 (Vcc), U?.20 (Vcc), U?.20 (Vcc), U?.20 (Vcc), U?.20 (Vcc), U?.20 (Vcc), U?.20 (Vcc), J?.2 (Vcc), U?.14 (VCC), U?.14 (VCC), U?.14 (VCC), U?.14 (VCC), U?.16 (VCC), U?.16 (VCC), U?.16 (VCC), U?.16 (VDD), U?.20 (VCC), U?.20 (VCC), U?.20 (VCC), U?.20 (VCC), U?.20 (VCC), U?.20 (VCC), U?.20 (VCC), U?.20 (VCC), U?.20 (Vcc), U?.20 (Vcc), U?.20 (Vcc), U?.20 (Vcc), U?.20 (Vcc), U?.20 (Vcc), U?.20 (Vcc), U?.20 (Vcc), U?.20 (Vcc), U?.20 (Vcc), U?.20 (Vcc), U?.20 (Vcc), U?.20 (Vcc), U?.20 (Vcc), U?.20 (Vcc), U?.20 (Vcc), U?.20 (Vcc), U?.20 (Vcc), U?.20 (Vcc), U?.6 (E2), U?.6 (E2), U?.6 (E2)
- net at U?.18 (2Q), U?.3 (2D), U?.3 (2D)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: now also U?.3 (2D), U?.3 (2D), U?.3 (2D), U?.3 (2D) (x2)
- net at U?.17 (3Q), U?.4 (3D), U?.4 (3D)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: now also U?.4 (3D), U?.4 (3D), U?.4 (3D), U?.4 (3D) (x2)
- net at U?.16 (4Q), U?.5 (4D), U?.5 (4D)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: now also U?.5 (4D), U?.5 (4D), U?.5 (4D), U?.5 (4D) (x2)
- net at U?.15 (5Q), U?.6 (5D), U?.6 (5D)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: now also U?.6 (5D), U?.6 (5D), U?.6 (5D), U?.6 (5D) (x2)
- net at U?.14 (6Q), U?.7 (6D), U?.7 (6D)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: now also U?.7 (6D), U?.7 (6D), U?.7 (6D), U?.7 (6D) (x2)
- net at U?.13 (7Q), U?.8 (7D), U?.8 (7D)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: now also U?.8 (7D), U?.8 (7D), U?.8 (7D), U?.8 (7D) (x2)
- net at U?.12 (8Q), U?.9 (8D), U?.9 (8D)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: now also U?.9 (8D), U?.9 (8D), U?.9 (8D), U?.9 (8D)
- net at U?.12 (8Q), U?.9 (8D), U?.9 (8D)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: now also U?.4, U?.5, U?.9, U?.9 (8D), U?.9 (8D), U?.9 (8D)
- net at U?.11 (LE): now also U?.11 (LE), U?.3 (x2)
- net at U?.2 (1D): now also J?.9 (Pin_9); no longer J?.1 (Pin_1)
- net at U?.3 (2D): now also J?.10 (Pin_10); no longer J?.2 (Pin_2)
- net at U?.4 (3D): now also J?.11 (Pin_11); no longer J?.3 (Pin_3)
- net at U?.5 (4D): now also J?.12 (Pin_12); no longer J?.4 (Pin_4)
- net at U?.6 (5D): now also J?.13 (Pin_13); no longer J?.5 (Pin_5)
- net at U?.7 (6D): now also J?.14 (Pin_14); no longer J?.6 (Pin_6)
- net at U?.8 (7D): now also J?.15 (Pin_15); no longer J?.7 (Pin_7)
- net at U?.9 (8D): now also J?.16 (Pin_16); no longer J?.8 (Pin_8)
- net at U?.2 (1D): now also J?.1 (Pin_1); no longer J?.9 (Pin_9)
- net at U?.3 (2D): now also J?.2 (Pin_2); no longer J?.10 (Pin_10)
- net at U?.4 (3D): now also J?.3 (Pin_3); no longer J?.11 (Pin_11)
- net at U?.5 (4D): now also J?.4 (Pin_4); no longer J?.12 (Pin_12)
- net at U?.6 (5D): now also J?.5 (Pin_5); no longer J?.13 (Pin_13)
- net at U?.7 (6D): now also J?.6 (Pin_6); no longer J?.14 (Pin_14)
- net at U?.8 (7D): now also J?.7 (Pin_7); no longer J?.15 (Pin_15)
- net at U?.9 (8D): now also J?.8 (Pin_8); no longer J?.16 (Pin_16)
- net at U?.1 (~G1): now also U?.1 (~G1), U?.15 (~Y0) (x2)
- net at U?.11 (Y8), U?.11 (Y8), U?.11 (Y8)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: now also J?.8 (Pin_8), U?.11 (Y8), U?.11 (Y8), U?.11 (Y8), U?.11 (Y8); no longer J?.8 (Pin_8)
- net at U?.12 (Y7), U?.12 (Y7), U?.12 (Y7)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: now also J?.7 (Pin_7), U?.12 (Y7), U?.12 (Y7), U?.12 (Y7), U?.12 (Y7); no longer J?.7 (Pin_7)
- net at U?.13 (Y6), U?.13 (Y6), U?.13 (Y6)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: now also J?.6 (Pin_6), U?.13 (Y6), U?.13 (Y6), U?.13 (Y6), U?.13 (Y6); no longer J?.6 (Pin_6)
- net at U?.14 (Y5), U?.14 (Y5), U?.14 (Y5)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: now also J?.5 (Pin_5), U?.14 (Y5), U?.14 (Y5), U?.14 (Y5), U?.14 (Y5); no longer J?.5 (Pin_5)
- net at U?.15 (Y4), U?.15 (Y4), U?.15 (Y4)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: now also J?.4 (Pin_4), U?.15 (Y4), U?.15 (Y4), U?.15 (Y4), U?.15 (Y4); no longer J?.4 (Pin_4)
- net at U?.16 (Y3), U?.16 (Y3), U?.16 (Y3)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: now also J?.3 (Pin_3), U?.16 (Y3), U?.16 (Y3), U?.16 (Y3), U?.16 (Y3); no longer J?.3 (Pin_3)
- net at U?.17 (Y2), U?.17 (Y2), U?.17 (Y2)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: now also J?.2 (Pin_2), U?.17 (Y2), U?.17 (Y2), U?.17 (Y2), U?.17 (Y2); no longer J?.2 (Pin_2)
- net at U?.18 (Y1), U?.18 (Y1), U?.18 (Y1)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: now also J?.1 (Pin_1), U?.18 (Y1), U?.18 (Y1), U?.18 (Y1), U?.18 (Y1); no longer J?.1 (Pin_1)
- net at U?.19 (~G2): now also U?.19 (~G2), U?.19 (~G2), U?.19 (~G2), U?.19 (~G2), U?.19 (~G2), U?.19 (~G2), U?.19 (~G2), U?.19 (~G2), U?.19 (~G2), U?.19 (~G2), U?.19 (~G2), U?.19 (~G2), U?.19 (~G2), U?.19 (~G2), U?.19 (~G2) (x2)
- net at U?.11 (Y8), U?.11 (Y8), U?.11 (Y8)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: now also J?.16 (Pin_16), U?.11 (Y8), U?.11 (Y8), U?.11 (Y8), U?.11 (Y8); no longer J?.16 (Pin_16)
- net at U?.12 (Y7), U?.12 (Y7), U?.12 (Y7)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: now also J?.15 (Pin_15), U?.12 (Y7), U?.12 (Y7), U?.12 (Y7), U?.12 (Y7); no longer J?.15 (Pin_15)
- net at U?.13 (Y6), U?.13 (Y6), U?.13 (Y6)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: now also J?.14 (Pin_14), U?.13 (Y6), U?.13 (Y6), U?.13 (Y6), U?.13 (Y6); no longer J?.14 (Pin_14)
- net at U?.14 (Y5), U?.14 (Y5), U?.14 (Y5)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: now also J?.13 (Pin_13), U?.14 (Y5), U?.14 (Y5), U?.14 (Y5), U?.14 (Y5); no longer J?.13 (Pin_13)
- net at U?.15 (Y4), U?.15 (Y4), U?.15 (Y4)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: now also J?.12 (Pin_12), U?.15 (Y4), U?.15 (Y4), U?.15 (Y4), U?.15 (Y4); no longer J?.12 (Pin_12)
- net at U?.16 (Y3), U?.16 (Y3), U?.16 (Y3)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: now also J?.11 (Pin_11), U?.16 (Y3), U?.16 (Y3), U?.16 (Y3), U?.16 (Y3); no longer J?.11 (Pin_11)
- net at U?.17 (Y2), U?.17 (Y2), U?.17 (Y2)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: now also J?.10 (Pin_10), U?.17 (Y2), U?.17 (Y2), U?.17 (Y2), U?.17 (Y2); no longer J?.10 (Pin_10)
- net at U?.18 (Y1), U?.18 (Y1), U?.18 (Y1)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: now also J?.9 (Pin_9), U?.18 (Y1), U?.18 (Y1), U?.18 (Y1), U?.18 (Y1); no longer J?.9 (Pin_9)
- net at U?.11 (Y8), U?.11 (Y8), U?.11 (Y8)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: now also J?.8 (Pin_8), U?.11 (Y8), U?.11 (Y8), U?.11 (Y8), U?.11 (Y8), U?.11 (Y8); no longer J?.8 (Pin_8)
- net at U?.12 (Y7), U?.12 (Y7), U?.12 (Y7)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: now also J?.7 (Pin_7), U?.12 (Y7), U?.12 (Y7), U?.12 (Y7), U?.12 (Y7), U?.12 (Y7); no longer J?.7 (Pin_7)
- net at U?.13 (Y6), U?.13 (Y6), U?.13 (Y6)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: now also J?.6 (Pin_6), U?.13 (Y6), U?.13 (Y6), U?.13 (Y6), U?.13 (Y6), U?.13 (Y6); no longer J?.6 (Pin_6)
- net at U?.14 (Y5), U?.14 (Y5), U?.14 (Y5)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: now also J?.5 (Pin_5), U?.14 (Y5), U?.14 (Y5), U?.14 (Y5), U?.14 (Y5), U?.14 (Y5); no longer J?.5 (Pin_5)
- net at U?.15 (Y4), U?.15 (Y4), U?.15 (Y4)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: now also J?.4 (Pin_4), U?.15 (Y4), U?.15 (Y4), U?.15 (Y4), U?.15 (Y4), U?.15 (Y4); no longer J?.4 (Pin_4)
- net at U?.16 (Y3), U?.16 (Y3), U?.16 (Y3)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: now also J?.3 (Pin_3), U?.16 (Y3), U?.16 (Y3), U?.16 (Y3), U?.16 (Y3), U?.16 (Y3); no longer J?.3 (Pin_3)
- net at U?.17 (Y2), U?.17 (Y2), U?.17 (Y2)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: now also J?.2 (Pin_2), U?.17 (Y2), U?.17 (Y2), U?.17 (Y2), U?.17 (Y2), U?.17 (Y2); no longer J?.2 (Pin_2)
- net at U?.18 (Y1), U?.18 (Y1), U?.18 (Y1)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: now also J?.1 (Pin_1), U?.18 (Y1), U?.18 (Y1), U?.18 (Y1), U?.18 (Y1), U?.18 (Y1); no longer J?.1 (Pin_1)
- net at U?.11 (Y8), U?.11 (Y8), U?.11 (Y8)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: now also J?.16 (Pin_16), U?.11 (Y8), U?.11 (Y8), U?.11 (Y8), U?.11 (Y8), U?.11 (Y8); no longer J?.16 (Pin_16)
- net at U?.12 (Y7), U?.12 (Y7), U?.12 (Y7)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: now also J?.15 (Pin_15), U?.12 (Y7), U?.12 (Y7), U?.12 (Y7), U?.12 (Y7), U?.12 (Y7); no longer J?.15 (Pin_15)
- net at U?.13 (Y6), U?.13 (Y6), U?.13 (Y6)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: now also J?.14 (Pin_14), U?.13 (Y6), U?.13 (Y6), U?.13 (Y6), U?.13 (Y6), U?.13 (Y6); no longer J?.14 (Pin_14)
- net at U?.14 (Y5), U?.14 (Y5), U?.14 (Y5)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: now also J?.13 (Pin_13), U?.14 (Y5), U?.14 (Y5), U?.14 (Y5), U?.14 (Y5), U?.14 (Y5); no longer J?.13 (Pin_13)
- net at U?.15 (Y4), U?.15 (Y4), U?.15 (Y4)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: now also J?.12 (Pin_12), U?.15 (Y4), U?.15 (Y4), U?.15 (Y4), U?.15 (Y4), U?.15 (Y4); no longer J?.12 (Pin_12)
- net at U?.16 (Y3), U?.16 (Y3), U?.16 (Y3)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: now also J?.11 (Pin_11), U?.16 (Y3), U?.16 (Y3), U?.16 (Y3), U?.16 (Y3), U?.16 (Y3); no longer J?.11 (Pin_11)
- net at U?.17 (Y2), U?.17 (Y2), U?.17 (Y2)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: now also J?.10 (Pin_10), U?.17 (Y2), U?.17 (Y2), U?.17 (Y2), U?.17 (Y2), U?.17 (Y2); no longer J?.10 (Pin_10)
- net at U?.18 (Y1), U?.18 (Y1), U?.18 (Y1)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: now also J?.9 (Pin_9), U?.18 (Y1), U?.18 (Y1), U?.18 (Y1), U?.18 (Y1), U?.18 (Y1); no longer J?.9 (Pin_9)
- net at U?.1 (~OE): now also U?.1 (~OE), U?.1 (~OE), U?.1 (~OE), U?.1 (~OE), U?.1 (~OE), U?.1 (~OE), U?.1 (~OE), U?.1 (~OE), U?.1 (~OE), U?.1 (~OE), U?.1 (~OE), U?.1 (~OE), U?.1 (~OE)
- net at U?.11 (LE): now also U?.11 (LE), U?.8
- net at U?.12 (8Q), U?.9 (A8), U?.9 (A8): now also J?.8 (Pin_8)
- net at U?.13 (7Q), U?.8 (A7), U?.8 (A7): now also J?.7 (Pin_7)
- net at U?.14 (6Q), U?.7 (A6), U?.7 (A6): now also J?.6 (Pin_6)
- net at U?.15 (5Q), U?.6 (A5), U?.6 (A5): now also J?.5 (Pin_5)
- net at U?.16 (4Q), U?.5 (A4), U?.5 (A4): now also J?.4 (Pin_4)
- net at U?.17 (3Q), U?.4 (A3), U?.4 (A3): now also J?.3 (Pin_3)
- net at U?.18 (2Q), U?.3 (A2), U?.3 (A2): now also J?.2 (Pin_2)
- net at U?.19 (1Q), U?.2 (A1), U?.2 (A1): now also J?.1 (Pin_1)
- net at U?.12 (8Q), U?.9 (A8), U?.9 (A8): now also J?.16 (Pin_16)
- net at U?.13 (7Q), U?.8 (A7), U?.8 (A7): now also J?.15 (Pin_15)
- net at U?.14 (6Q), U?.7 (A6), U?.7 (A6): now also J?.14 (Pin_14)
- net at U?.15 (5Q), U?.6 (A5), U?.6 (A5): now also J?.13 (Pin_13)
- net at U?.16 (4Q), U?.5 (A4), U?.5 (A4): now also J?.12 (Pin_12)
- net at U?.17 (3Q), U?.4 (A3), U?.4 (A3): now also J?.11 (Pin_11)
- net at U?.18 (2Q), U?.3 (A2), U?.3 (A2): now also J?.10 (Pin_10)
- net at U?.19 (1Q), U?.2 (A1), U?.2 (A1): now also J?.9 (Pin_9)
- net at U?.1 (~G1): now also U?.1 (~G1), U?.14 (~Y1) (x2)
- net at U?.11 (LE): now also U?.11 (LE), U?.11
- net at U?.1 (~G1): now also U?.1 (~G1), U?.13 (~Y2) (x2)
- net at U?.1 (~G1): now also U?.1 (~G1), U?.12 (~Y3) (x2)
- new net: U?.11 (LE), U?.11 (LE), U?.6
- new net: U?.12 (8Q), U?.9 (A8), U?.9 (A8) (x6)
- new net: U?.13 (7Q), U?.8 (A7), U?.8 (A7) (x6)
- new net: U?.14 (6Q), U?.7 (A6), U?.7 (A6) (x6)
- new net: U?.15 (5Q), U?.6 (A5), U?.6 (A5) (x6)
- new net: U?.16 (4Q), U?.5 (A4), U?.5 (A4) (x6)
- new net: U?.17 (3Q), U?.4 (A3), U?.4 (A3) (x6)
- new net: U?.18 (2Q), U?.3 (A2), U?.3 (A2) (x6)
- new net: U?.19 (1Q), U?.2 (A1), U?.2 (A1) (x6)
- new net: U?.1 (~G1), U?.1 (~G1), U?.11 (~Y4) (x2)
- new net: U?.11 (LE), U?.11 (LE), U?.8
- new net: U?.1 (~G1), U?.1 (~G1), U?.10 (~Y5) (x2)
- new net: U?.11, U?.11 (LE), U?.11 (LE)
- new net: U?.1 (~G1), U?.1 (~G1), U?.9 (~Y6) (x2)
- new net: U?.10, U?.11 (LE), U?.11 (LE), U?.12, U?.6
- new net: J?.8 (Pin_8), U?.12 (8Q), U?.9 (A8), U?.9 (A8)
- new net: J?.7 (Pin_7), U?.13 (7Q), U?.8 (A7), U?.8 (A7)
- new net: J?.6 (Pin_6), U?.14 (6Q), U?.7 (A6), U?.7 (A6)
- new net: J?.5 (Pin_5), U?.15 (5Q), U?.6 (A5), U?.6 (A5)
- new net: J?.4 (Pin_4), U?.16 (4Q), U?.5 (A4), U?.5 (A4)
- new net: J?.3 (Pin_3), U?.17 (3Q), U?.4 (A3), U?.4 (A3)
- new net: J?.2 (Pin_2), U?.18 (2Q), U?.3 (A2), U?.3 (A2)
- new net: J?.1 (Pin_1), U?.19 (1Q), U?.2 (A1), U?.2 (A1)
- new net: J?.15 (Pin_15), U?.13 (7Q), U?.8 (A7), U?.8 (A7)
- new net: J?.14 (Pin_14), U?.14 (6Q), U?.7 (A6), U?.7 (A6)
- new net: J?.13 (Pin_13), U?.15 (5Q), U?.6 (A5), U?.6 (A5)
- new net: J?.12 (Pin_12), U?.16 (4Q), U?.5 (A4), U?.5 (A4)
- new net: J?.11 (Pin_11), U?.17 (3Q), U?.4 (A3), U?.4 (A3)
- new net: J?.10 (Pin_10), U?.18 (2Q), U?.3 (A2), U?.3 (A2)
- new net: J?.9 (Pin_9), U?.19 (1Q), U?.2 (A1), U?.2 (A1)
- new net: U?.1 (~G1), U?.1 (~G1), U?.7 (~Y7) (x2)
- new net: J?.16 (Pin_16), U?.1 (Q), U?.4, U?.9 (A8), U?.9 (A8)
- new net: J?.1 (Pin_1), U?.2 (A1)
- new net: J?.10 (Pin_10), U?.3 (A2)
- new net: J?.11 (Pin_11), U?.4 (A3)
- new net: J?.12 (Pin_12), U?.5 (A4)
- new net: J?.13 (Pin_13), U?.6 (A5)
- new net: J?.14 (Pin_14), U?.7 (A6)
- new net: J?.15 (Pin_15), U?.8 (A7)
- new net: J?.16 (Pin_16), U?.9 (A8)
- new net: J?.2 (Pin_2), U?.3 (A2)
- new net: J?.3 (Pin_3), U?.4 (A3)
- new net: J?.4 (Pin_4), U?.5 (A4)
- new net: J?.5 (Pin_5), U?.6 (A5)
- new net: J?.6 (Pin_6), U?.7 (A6)
- new net: J?.7 (Pin_7), U?.8 (A7)
- new net: J?.8 (Pin_8), U?.9 (A8)
- new net: J?.9 (Pin_9), U?.2 (A1)
- new net: U?.1 (~G1), U?.1 (~G1), U?.3
- new net: J?.4 (CLK_F), U?.3 (C), U?.5
- new net: U?.11, U?.4 (R)
- new net: U?.7 (S), U?.8
- new net: U?.13, U?.6
- new net: J?.3 (Pin_3), U?.1 (A0) (x3)
- new net: J?.2 (Pin_2), U?.2 (A1) (x3)
- new net: J?.1 (Pin_1), U?.3 (A2) (x3)
- new net: U?.10 (~Y5), U?.7 (A6)
- new net: U?.11 (~Y4), U?.6 (A5)
- new net: U?.12 (~Y3), U?.5 (A4)
- new net: U?.13 (~Y2), U?.4 (A3)
- new net: U?.14 (~Y1), U?.3 (A2)
- new net: U?.15 (~Y0), U?.2 (A1)
- new net: U?.7 (~Y7), U?.9 (A8)
- new net: U?.8 (A7), U?.9 (~Y6)
- new net: U?.1 (~G1), U?.19 (~G2)
- new net: U?.1, U?.11 (~Y8)
- new net: U?.12 (~Y7), U?.13
- new net: U?.10, U?.13 (~Y6)
- new net: U?.14 (~Y5), U?.5
- new net: U?.15 (~Y4), U?.2
- new net: U?.13, U?.16 (~Y3)
- new net: U?.10, U?.17 (~Y2)
- new net: J?.3 (CLK_R), U?.2
- new net: U?.1, U?.12, U?.12, U?.2, U?.4, U?.6, U?.9, U?.9
- new net: U?.3, U?.5
- new net Const_Reg: J?.3 (Pin_3), U?.1, U?.2, U?.5 (~E1)
- new net R_Sup: J?.2 (Pin_2), U?.5 (K)
- new net S_Sup: J?.1 (Pin_1), U?.6 (J)
- new net WE: J?.5 (Pin_5), U?.1, U?.4
Other:
- note added: "A"
- note added: "B"
- note added: "C"
- note added: "D"
- note added: "FLAG"
- note added: "IP"
- note added: "SP"
- note added: "ZERO"
- moved on the sheet: J?, U?
