File: circets/Register_File/register_file_kicad/register_file_kicad.sch (KiCad schematic (older format))
At the start: 85 parts

Commit message: Fixed Issue with wrong pins in activation Module!
Parts:
- J?: symbol Computer_Component_Library:Bus_Connector -> register_file_kicad-rescue:Bus_Connector-Computer_Component_Library
Changed lines of the file:
@@
 	7900 12950 7900 13200
 $Comp
-L Computer_Component_Library:Bus_Connector J?
+L register_file_kicad-rescue:Bus_Connector-Computer_Component_Library J?
 U 1 1 F4535150
 P 4050 900
