File: circets/Register_File/register_file_kicad/register_file_kicad.kicad_pcb (KiCad board)
At the start: 2 copper layers, 356.5 x 331.7 mm, 92 parts, among them J1 A_Out, J10 Conn_01x16_Male, J11 Const_In, J12 Flag_Out, J13 Conn_01x16_Female, J14 Conn_01x12_Male, J15 Conn_01x12_Female, J2 B_Out, J3 D_Sel, J4 AM-Connector, J5 Conn_01x04_Female, J6 Bus_Connector, J7 B_Sel, J8 A_Sel, J9 Conn_01x16_Female, U1 74LS32, U10 74HC541, U11 74HC283, U12 74HC573, U13 74LS08, U14 74HC541, U15 74HC541, U16 74HC137, U17 74HC137, U18 74HC573, U19 74HC283, U2 SRGB_Bar_2000, U20 74HC541, U21 74HC541, U22 74HC573, U23 74HC283, U24 74LS08, U25 74HC541, U26 74HC541, U27 74LS08, U28 74HC573, U29 74HC00, U3 SRGB_Bar_2000, U30 4027, U31 74HC541, U32 74HC541, U33 74HC573, U34 74HC541, U35 74HC541, U36 74HC573, U37 74HC541, U38 74HC541, U39 74HC573, U4 74HC137, U40 74HC541, U41 74HC541, U42 74HC573, U43 74HC541, U44 74HC541, U45 74HC573, U46 74HC541, U47 74HC541, U48 74HC573, U49 74HC541, U5 74HC283, U50 74HC541, U51 74HC573, U52 74HC541, U53 74HC541, U54 74HC573, U55 74HC541, U56 74HC541, U57 74HC573, U58 74HC541, U59 74HC541, U6 74HC540, U60 74HC573, U61 74HC541, U62 74HC541, U63 74HC541, U64 74HC573, U65 74HC541, U66 74HC541, U67 74HC541, U68 74LS00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

Commit message: Did **Something** to the file by apperently not editing it, idk
Parts:
- moved U6 8.88 mm to (143.0, 77.7)
Changed lines of the file:
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@@
   )
   (footprint "Package_DIP:DIP-20_W7.62mm_Socket" (layer "F.Cu")
-    (at 138.954 85.632)
+    (at 143.012 77.729)
     (descr "20-lead though-hole mounted DIP package, row spacing 7.62 mm (300 mils), Socket")
     (tags "THT DIP DIL PDIP 2.54mm 7.62mm 300mil Socket")

Commit message: Added Siwas Register File PCB + compleateted it!
Parts:
- removed the U29 at (108.2, 84.5)
- added J16: Conn_01x01_Female, Connector_PinSocket_2.54mm:PinSocket_1x01_P2.54mm_Vertical, F.Cu at (407.8, 52.9)
- added J17: Conn_01x01_Female, Connector_PinSocket_2.54mm:PinSocket_1x01_P2.54mm_Vertical, F.Cu at (130.3, 211.3)
- added J18: Sup_Conn_main, Connector_PinSocket_2.54mm:PinSocket_1x03_P2.54mm_Horizontal, F.Cu at (36.3, 202.4)
- added J19: Sup_Conn_Sec, Connector_PinSocket_2.54mm:PinSocket_1x03_P2.54mm_Horizontal, F.Cu at (407.9, 43.3)
- J3: footprint Connector_PinHeader_2.54mm:PinHeader_1x16_P2.54mm_Vertical -> Connector_PinSocket_2.54mm:PinSocket_1x03_P2.54mm_Horizontal
- U10, U9: footprint Package_DIP:DIP-20_W7.62mm_Socket -> Package_SO:SO-20_5.3x12.6mm_P1.27mm
- U14, U15, U20, U21, U25, U26, U31, U32, U34, U35, U37, U38, U40, U41, U43, U44, U46, U47, U49, U50, U52, U53, U55, U56, U58, U59, U61, U62, U63, U65, U66, U67: footprint Package_DIP:DIP-20_W7.62mm_Socket -> Package_SO:SO-20_12.8x7.5mm_P1.27mm
- moved R6 421.3 mm to (494.8, 98.2), turned to 180 degrees
- moved U12 405.7 mm to (459.0, 111.0), turned to -90 degrees
- moved R5 400.9 mm to (494.8, 102.2), turned to 180 degrees
- moved U23 398.4 mm to (480.7, 57.7), turned to 0 degrees
- moved J3 394.4 mm to (523.8, 45.5), turned to 90 degrees
- moved U4 386.4 mm to (518.9, 42.3), turned to -90 degrees
- moved J4 385.9 mm to (420.2, 91.2), turned to 90 degrees
- moved U19 385.1 mm to (467.9, 57.8), turned to 0 degrees
- moved U8 384.3 mm to (459.1, 98.7)
- moved U30 382.8 mm to (489.1, 34.9), turned to -90 degrees
- moved R7 380.6 mm to (506.0, 36.4), turned to 180 degrees
- moved U7 379.7 mm to (429.9, 111.0), turned to -90 degrees
- moved D1 377.5 mm to (497.1, 37.4), turned to 180 degrees
- moved U6 376.6 mm to (518.9, 55.3), turned to -90 degrees
- moved J10 373.9 mm to (405.2, 123.7), turned to -90 degrees
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Connections:
- J14 pad 12: unconnected-(J14-Pad12) -> /Zero_One
- J15 pad 12: unconnected-(J15-Pad12) -> Net-(J15-Pad12)
- J6 pad 65: Net-(D1-Pad2) -> Net-(J6-Pad65)
- J6 pad 66: S_Sup -> Net-(J6-Pad66)
- J6 pad 67: R_Sup -> Net-(J6-Pad67)
- U10 pad 2: /Zero_One -> Net-(J15-Pad12)
- U16 pad 5: /Const_Reg -> Net-(U16-Pad5)
- U29 pad 1: /Const_Reg -> Net-(U16-Pad5)
- U29 pad 2: /Const_Reg -> Net-(U16-Pad5)
- U9 pad 2: /Zero_One -> Net-(J15-Pad12)
Routing:
- net Net-(U10-Pad3): track 1533.1 -> 194.1 mm, vias 32 -> 4
- net GND: track 3267.7 -> 3990.9 mm, vias 23 -> 38
- net +5V: track 1329.9 -> 1925.2 mm, vias 16 -> 56
- net Net-(J13-Pad5): track 533.8 -> 0.00 mm, vias 7 -> 0
- net Net-(J13-Pad6): track 549.3 -> 1077.8 mm, vias 7 -> 14
- net Net-(J13-Pad9): track 403.8 -> 0.00 mm, vias 7 -> 0
- net Net-(U17-Pad7): track 289.0 -> 0.00 mm, vias 2 -> 0
- net Net-(J14-Pad2): track 0.00 -> 180.7 mm, vias 0 -> 4
- net Net-(J14-Pad6): track 0.00 -> 178.0 mm, vias 0 -> 2
- net Net-(J14-Pad5): track 0.00 -> 166.8 mm, vias 0 -> 1
- net Net-(D1-Pad2): track 0.00 -> 163.7 mm, vias 0 -> 7
- net Net-(J14-Pad3): track 0.00 -> 159.3 mm, vias 0 -> 2
- net Net-(J14-Pad4): track 0.00 -> 155.8 mm
- net Net-(J14-Pad8): track 0.00 -> 149.9 mm, vias 0 -> 2
- net Net-(J4-Pad26): track 163.4 -> 26.5 mm, vias 5 -> 0
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Other:
- board size 356.5 x 331.7 mm -> 505.4 x 180.6 mm
- board text added: "Memory primary"
- board text added: "Memory secondary"

Commit message: fixed all design-issues in register_file
Parts:
- moved U45 0.62 mm to (241.1, 82.7)
- moved J10 0.60 mm to (405.8, 123.7)
- moved J13 0.56 mm to (37.0, 44.9)
- moved U33 0.52 mm to (160.5, 82.6)
- moved U32 0.46 mm to (137.2, 153.3)
- moved U51 0.29 mm to (281.6, 82.7)
- moved U28 0.28 mm to (140.7, 82.6)
- moved J15 0.11 mm to (35.7, 41.2)
- moved U22 0.10 mm to (119.9, 82.6)
- moved U39 0.07 mm to (200.8, 82.7)
- moved U18 0.06 mm to (100.0, 82.6)
Routing:
- net Net-(J13-Pad5): track 0.00 -> 535.2 mm, vias 0 -> 7
- net Net-(J13-Pad6): track 1077.8 -> 543.1 mm, vias 14 -> 7
- net Net-(J13-Pad9): track 0.00 -> 403.2 mm, vias 0 -> 7
- net GND: track 3990.9 -> 3632.7 mm, vias 38 -> 32
- net Net-(U17-Pad7): track 0.00 -> 294.0 mm, vias 0 -> 2
- net +5V: track 1925.2 -> 1647.4 mm, vias 56 -> 55
- net Net-(J14-Pad1): track 0.00 -> 184.0 mm, vias 0 -> 2
- net Net-(U12-Pad11): track 0.00 -> 178.1 mm, vias 0 -> 3
- net Net-(U1-Pad10): track 0.00 -> 48.0 mm, vias 0 -> 2
- net Net-(R1-Pad2): track 58.2 -> 21.7 mm
- net Net-(U16-Pad10): track 321.9 -> 299.9 mm
- net Net-(R3-Pad2): track 0.00 -> 21.5 mm
- net Net-(U16-Pad14): track 159.3 -> 138.5 mm
- net Net-(U27-Pad5): track 0.00 -> 20.5 mm
- net Net-(J12-Pad1): track 169.4 -> 153.5 mm
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Other:
- board size 505.4 x 180.6 mm -> 505.4 x 181.7 mm

Commit message: Changed Label on Register File
Parts:
- added J20: Conn_01x02_Female, Connector_PinSocket_2.54mm:PinSocket_1x02_P2.54mm_Vertical, F.Cu at (36.5, 37.1)
- added J21: Conn_01x02_Female, Connector_PinSocket_2.54mm:PinSocket_1x02_P2.54mm_Vertical, F.Cu at (439.0, 155.8)
- moved U1 113.6 mm to (528.0, 38.5), turned to -90 degrees
- moved J19 113.4 mm to (520.7, 32.0), turned to 180 degrees
- moved J14 105.7 mm to (438.4, 26.3), turned to -90 degrees
- moved J16 105.4 mm to (511.1, 32.0), turned to 0 degrees
- moved J5 103.4 mm to (498.0, 26.5), turned to 0 degrees
- moved J3 102.6 mm to (518.5, 148.0), turned to 0 degrees
- moved U4 100.8 mm to (521.7, 143.0), turned to 180 degrees
- moved J10 99.9 mm to (440.3, 29.9), turned to 180 degrees
- moved R7 96.2 mm to (527.6, 130.1), turned to 90 degrees
- moved U68 91.8 mm to (529.2, 67.5), turned to 180 degrees
- moved D1 88.9 mm to (526.6, 121.3), turned to 90 degrees
- moved U6 88.3 mm to (508.7, 143.1), turned to 180 degrees
- moved U30 88.0 mm to (529.2, 113.2), turned to 180 degrees
- moved U27 84.1 mm to (529.2, 89.0), turned to 180 degrees
- moved J4 76.6 mm to (471.5, 34.3), turned to 0 degrees
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Connections:
- U13 pad 2: Net-(J6-Pad3) -> Net-(U13-Pad2)
- U13 pad 5: Net-(J6-Pad4) -> Net-(U13-Pad5)
Routing:
- net GND: track 3632.7 -> 3566.1 mm
- net Net-(U13-Pad2): track 0.00 -> 63.0 mm, vias 0 -> 1
- net Net-(U13-Pad5): track 0.00 -> 60.2 mm, vias 0 -> 2
- net +5V: track 1647.4 -> 1697.3 mm, vias 55 -> 56
- net Net-(J15-Pad12): track 131.7 -> 172.4 mm
- net Net-(U12-Pad3): track 91.2 -> 118.6 mm, vias 0 -> 2
- net Net-(U12-Pad4): track 109.4 -> 136.1 mm, vias 0 -> 2
- net Net-(U11-Pad1): track 104.4 -> 130.7 mm, vias 0 -> 4
- net Net-(U11-Pad13): track 121.8 -> 148.1 mm, vias 0 -> 2
- net Net-(U11-Pad10): track 130.4 -> 156.7 mm, vias 0 -> 2
- net Net-(U11-Pad4): track 111.6 -> 137.4 mm, vias 0 -> 4
- net Net-(J2-Pad16): track 712.3 -> 686.6 mm
- net Net-(U12-Pad5): track 118.1 -> 143.3 mm, vias 0 -> 2
- net Net-(J6-Pad4): track 0.00 -> 20.5 mm
- net Net-(U12-Pad2): track 88.8 -> 109.1 mm, vias 0 -> 2
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Other:
- board size 505.4 x 181.7 mm -> 503.1 x 191.5 mm
