File: circets/Register_File/register_file_kicad/register_file_kicad.kicad_sch (KiCad schematic)
At the start: 85 parts

Commit message: Build Register File PCB-Layout
Parts:
- removed J?: D_In, symbol Connector:Conn_01x16_Female
- removed J?: Conn_01x05_Female, symbol Connector:Conn_01x05_Female
- removed J?: Bus_Connector, symbol register_file_kicad-rescue:Bus_Connector-Computer_Component_Library
- removed U?: 74HC00, symbol 74xx:74HC00
- added D1: LED, LED_THT:LED_D5.0mm, symbol Device:LED
- added J10: Conn_01x16_Male, Connector_PinSocket_2.54mm:PinSocket_1x16_P2.54mm_Vertical, symbol Connector:Conn_01x16_Male
- added J13: Conn_01x16_Female, Connector_PinSocket_2.54mm:PinSocket_1x16_P2.54mm_Vertical, symbol Connector:Conn_01x16_Female
- added J14: Conn_01x12_Male, Connector_PinSocket_2.54mm:PinSocket_1x12_P2.54mm_Vertical, symbol Connector:Conn_01x12_Male
- added J15: Conn_01x12_Female, Connector_PinSocket_2.54mm:PinSocket_1x12_P2.54mm_Vertical, symbol Connector:Conn_01x12_Female
- added J4: AM-Connector, Computer_Component_Library:PinHeader_1x42_P2.54mm_Horizontal, symbol Computer_Component_Library:AM-Connector
- added J5: Conn_01x04_Female, Connector_PinHeader_2.54mm:PinHeader_1x04_P2.54mm_Horizontal, symbol Connector:Conn_01x04_Female
- added J6: Bus_Connector, Computer_Component_Library:PinHeader_1x78_P2.54mm_Horizontal, symbol Computer_Component_Library:Bus_Connector
- added R1, R2, R3, R4, R5, R6, R7: 220, Resistor_THT:R_Axial_DIN0309_L9.0mm_D3.2mm_P5.08mm_Vertical, symbol Device:R
- added U1: 74LS32, Package_DIP:DIP-14_W7.62mm_Socket, symbol 74xx:74LS32
- added U11, U19, U23, U5: 74HC283, Package_DIP:DIP-16_W7.62mm_Socket, symbol Custome_Components:74HC283
- added U2, U3, U8: SRGB_Bar_2000, Computer_Component_Library:SRGB_2000, symbol Computer_Component_Library:SRGB_Bar_2000
- added U68: 74LS00, Package_DIP:DIP-14_W7.62mm_Socket, symbol 74xx:74LS00
- J1, J2, J3: renamed from J?; footprint (none) -> Connector_PinHeader_2.54mm:PinHeader_1x16_P2.54mm_Vertical
- J11, J12: renamed from J?; footprint (none) -> Connector_PinHeader_2.54mm:PinHeader_1x16_P2.54mm_Horizontal
- J7, J8: renamed from J?; footprint (none) -> Connector_PinHeader_2.54mm:PinHeader_1x03_P2.54mm_Horizontal
- J9: renamed from J?; footprint (none) -> Connector_PinSocket_2.54mm:PinSocket_1x16_P2.54mm_Vertical
- U10, U12, U14, U15, U18, U20, U21, U22, U25, U26, U28, U31, U32, U33, U34, U35, U36, U37, U38, U39, U40, U41, U42, U43, U44, U45, U46, U47, U48, U49, U50, U51, U52, U53, U54, U55, U56, U57, U58, U59, U6, U60, U61, U62, U63, U64, U65, U66, U67, U7, U9: renamed from U?; footprint (none) -> Package_DIP:DIP-20_W7.62mm_Socket
- U13, U24, U27, U29: renamed from U?; footprint (none) -> Package_DIP:DIP-14_W7.62mm_Socket
- U16, U17, U30, U4: renamed from U?; footprint (none) -> Package_DIP:DIP-16_W7.62mm_Socket
Connections:
- net +5V: now also J14.10 (Pin_10), J15.10 (Pin_10), J6.2 (Vcc), U1.14 (VCC), U11.16 (Vcc), U19.16 (Vcc), U23.16 (Vcc), U5.16 (Vcc), U68.14 (VCC)
- net Const_Reg: now also J5.3 (Pin_3)
- net GND: now also U10.19 (~{G2}), U12.1 (~{OE}), U14.19 (~{G2}), U15.19 (~{G2}), U18.1 (~{OE}), U20.19 (~{G2}), U21.19 (~{G2}), U22.1 (~{OE}), U25.19 (~{G2}), U26.19 (~{G2}), U28.1 (~{OE}), U30.3 (C), U30.5 (K), U30.6 (J), U31.19 (~{G2}), U32.19 (~{G2}), U33.1 (~{OE}), U34.19 (~{G2}), U35.19 (~{G2}), U36.1 (~{OE}), U37.19 (~{G2}), U38.19 (~{G2}), U39.1 (~{OE}), U40.19 (~{G2}), U41.19 (~{G2}), U42.1 (~{OE}), U43.19 (~{G2}), U44.19 (~{G2}), U45.1 (~{OE}), U46.19 (~{G2}), U47.19 (~{G2}), U48.1 (~{OE}), U49.19 (~{G2}), U50.19 (~{G2}), U51.1 (~{OE}), U52.19 (~{G2}), U53.19 (~{G2}), U54.1 (~{OE}), U55.19 (~{G2}), U56.19 (~{G2}), U57.1 (~{OE}), U58.19 (~{G2}), U59.19 (~{G2}), U60.1 (~{OE}), U61.19 (~{G2}), U62.19 (~{G2}), U63.19 (~{G2}), U64.1 (~{OE}), U65.19 (~{G2}), U66.19 (~{G2}), U67.19 (~{G2}), U7.1 (~{OE}), U9.19 (~{G2}), J14.11 (Pin_11), J15.11 (Pin_11), J6.1 (GND), R1.1, R2.1, R3.1, R4.1, R5.1, R6.1, R7.1, U1.7 (GND), U11.8 (GND), U19.8 (GND), U23.8 (GND), U5.7 (C0), U5.8 (GND), U68.7 (GND)
- net R_Sup: now also J6.67 (Reset_Sup), U1.9; no longer U30.5 (K)
- net S_Sup: now also J6.66 (Set_Sup), U1.4; no longer U30.6 (J)
- net WE: now also J4.9 (WE)
- net Zero_One: now also J5.4 (Pin_4)
- net at U42.11 (LE), U45.11 (LE): now also J15.4 (Pin_4); no longer U24.6
- net at U18.2 (1D), U28.2 (1D), U36.2 (1D)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: now also J13.16 (Pin_16); no longer U12.19 (1Q)
- net at U18.3 (2D), U28.3 (2D), U36.3 (2D)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: now also J13.15 (Pin_15); no longer U12.18 (2Q)
- net at U18.4 (3D), U28.4 (3D), U36.4 (3D)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: now also J13.14 (Pin_14); no longer U12.17 (3Q)
- net at U18.5 (4D), U28.5 (4D), U36.5 (4D)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: now also J13.13 (Pin_13); no longer U12.16 (4Q)
- net at U18.6 (5D), U28.6 (5D), U36.6 (5D)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: now also J13.12 (Pin_12); no longer U12.15 (5Q)
- net at U18.7 (6D), U28.7 (6D), U36.7 (6D)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: now also J13.11 (Pin_11); no longer U12.14 (6Q)
- net at U18.8 (7D), U28.8 (7D), U36.8 (7D)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: now also J13.10 (Pin_10); no longer U12.13 (7Q)
- net at U18.9 (8D), U28.9 (8D), U36.9 (8D)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: now also J13.9 (Pin_9); no longer U12.12 (8Q)
- net at U22.2 (1D), U33.2 (1D), U39.2 (1D)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: now also J13.8 (Pin_8); no longer U7.19 (1Q)
- net at U22.3 (2D), U33.3 (2D), U39.3 (2D)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: now also J13.7 (Pin_7); no longer U7.18 (2Q)
- net at U22.4 (3D), U33.4 (3D), U39.4 (3D)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: now also J13.6 (Pin_6); no longer U7.17 (3Q)
- net at U22.5 (4D), U33.5 (4D), U39.5 (4D)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: now also J13.5 (Pin_5); no longer U7.16 (4Q)
- net at U22.6 (5D), U33.6 (5D), U39.6 (5D)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: now also J13.4 (Pin_4); no longer U7.15 (5Q)
- net at U22.7 (6D), U33.7 (6D), U39.7 (6D)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: now also J13.3 (Pin_3); no longer U7.14 (6Q)
- net at U22.8 (7D), U33.8 (7D), U39.8 (7D)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: now also J13.2 (Pin_2); no longer U7.13 (7Q)
- net at U22.9 (8D), U33.9 (8D), U39.9 (8D)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: now also J13.1 (Pin_1), J15.7 (Pin_7); no longer U27.9, U7.12 (8Q)
- net at U20.11 (Y8), U31.11 (Y8), U37.11 (Y8)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: now also J1.8 (Pin_8), U2.9; no longer J2.8 (Pin_8)
- net at U20.12 (Y7), U31.12 (Y7), U37.12 (Y7)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: now also J1.7 (Pin_7), U2.10; no longer J2.7 (Pin_7)
- net at U20.13 (Y6), U31.13 (Y6), U37.13 (Y6)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: now also J1.6 (Pin_6), U2.11; no longer J2.6 (Pin_6)
- net at U20.14 (Y5), U31.14 (Y5), U37.14 (Y5)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: now also J1.5 (Pin_5), U2.12; no longer J2.5 (Pin_5)
- net at U20.15 (Y4), U31.15 (Y4), U37.15 (Y4)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: now also J1.4 (Pin_4), U2.13; no longer J2.4 (Pin_4)
- net at U20.16 (Y3), U31.16 (Y3), U37.16 (Y3)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: now also J1.3 (Pin_3), U2.14; no longer J2.3 (Pin_3)
- net at U20.17 (Y2), U31.17 (Y2), U37.17 (Y2)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: now also J1.2 (Pin_2), U2.15; no longer J2.2 (Pin_2)
- net at U20.18 (Y1), U31.18 (Y1), U37.18 (Y1)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: now also J1.1 (Pin_1), U2.16; no longer J2.1 (Pin_1)
- net at U14.11 (Y8), U25.11 (Y8), U34.11 (Y8)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: now also J1.16 (Pin_16), U2.1; no longer J2.16 (Pin_16)
- net at U14.12 (Y7), U25.12 (Y7), U34.12 (Y7)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: now also J1.15 (Pin_15), U2.2; no longer J2.15 (Pin_15)
- net at U14.13 (Y6), U25.13 (Y6), U34.13 (Y6)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: now also J1.14 (Pin_14), U2.3; no longer J2.14 (Pin_14)
- net at U14.14 (Y5), U25.14 (Y5), U34.14 (Y5)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: now also J1.13 (Pin_13), U2.4; no longer J2.13 (Pin_13)
- net at U14.15 (Y4), U25.15 (Y4), U34.15 (Y4)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: now also J1.12 (Pin_12), U2.5; no longer J2.12 (Pin_12)
- net at U14.16 (Y3), U25.16 (Y3), U34.16 (Y3)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: now also J1.11 (Pin_11), U2.6; no longer J2.11 (Pin_11)
- net at U14.17 (Y2), U25.17 (Y2), U34.17 (Y2)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: now also J1.10 (Pin_10), U2.7; no longer J2.10 (Pin_10)
- net at U14.18 (Y1), U25.18 (Y1), U34.18 (Y1)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: now also J1.9 (Pin_9), U2.8; no longer J2.9 (Pin_9)
- net at U10.11 (Y8), U21.11 (Y8), U32.11 (Y8)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: now also J2.8 (Pin_8), U3.9; no longer J1.8 (Pin_8)
- net at U10.12 (Y7), U21.12 (Y7), U32.12 (Y7)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: now also J2.7 (Pin_7), U3.10; no longer J1.7 (Pin_7)
- net at U10.13 (Y6), U21.13 (Y6), U32.13 (Y6)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: now also J2.6 (Pin_6), U3.11; no longer J1.6 (Pin_6)
- net at U10.14 (Y5), U21.14 (Y5), U32.14 (Y5)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: now also J2.5 (Pin_5), U3.12; no longer J1.5 (Pin_5)
- net at U10.15 (Y4), U21.15 (Y4), U32.15 (Y4)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: now also J2.4 (Pin_4), U3.13; no longer J1.4 (Pin_4)
- net at U10.16 (Y3), U21.16 (Y3), U32.16 (Y3)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: now also J2.3 (Pin_3), U3.14; no longer J1.3 (Pin_3)
- net at U10.17 (Y2), U21.17 (Y2), U32.17 (Y2)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: now also J2.2 (Pin_2), U3.15; no longer J1.2 (Pin_2)
- net at U10.18 (Y1), U21.18 (Y1), U32.18 (Y1)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: now also J2.1 (Pin_1), U3.16; no longer J1.1 (Pin_1)
- net at U15.11 (Y8), U26.11 (Y8), U35.11 (Y8)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: now also J2.16 (Pin_16), U3.1; no longer J1.16 (Pin_16)
- net at U15.12 (Y7), U26.12 (Y7), U35.12 (Y7)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: now also J2.15 (Pin_15), U3.2; no longer J1.15 (Pin_15)
- net at U15.13 (Y6), U26.13 (Y6), U35.13 (Y6)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: now also J2.14 (Pin_14), U3.3; no longer J1.14 (Pin_14)
- net at U15.14 (Y5), U26.14 (Y5), U35.14 (Y5)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: now also J2.13 (Pin_13), U3.4; no longer J1.13 (Pin_13)
- net at U15.15 (Y4), U26.15 (Y4), U35.15 (Y4)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: now also J2.12 (Pin_12), U3.5; no longer J1.12 (Pin_12)
- net at U15.16 (Y3), U26.16 (Y3), U35.16 (Y3)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: now also J2.11 (Pin_11), U3.6; no longer J1.11 (Pin_11)
- net at U15.17 (Y2), U26.17 (Y2), U35.17 (Y2)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: now also J2.10 (Pin_10), U3.7; no longer J1.10 (Pin_10)
- net at U15.18 (Y1), U26.18 (Y1), U35.18 (Y1)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: now also J2.9 (Pin_9), U3.8; no longer J1.9 (Pin_9)
- net at U48.11 (LE), U51.11 (LE): now also J15.5 (Pin_5); no longer U24.8
- net at U54.11 (LE), U57.11 (LE): now also J15.6 (Pin_6); no longer U24.11
- net at J12.16 (Pin_16), U65.9 (A8), U66.9 (A8): no longer U27.4, U30.1 (Q)
- net at U7.2 (1D): now also U19.4 (S1)
- net at U7.3 (2D): now also U19.1 (S2)
- net at U7.4 (3D): now also U19.13 (S3)
- net at U7.5 (4D): now also U19.10 (S4)
- net at U7.6 (5D): now also U23.4 (S1)
- net at U7.7 (6D): now also U23.1 (S2)
- net at U7.8 (7D): now also U23.13 (S3)
- net at U7.9 (8D): now also U23.10 (S4)
- net at U12.2 (1D): now also U5.4 (S1)
- net at U12.3 (2D): now also U5.1 (S2)
- net at U12.4 (3D): now also U5.13 (S3)
- net at U12.5 (4D): now also U5.10 (S4)
- net at U12.6 (5D): now also U11.4 (S1)
- net at U12.7 (6D): now also U11.1 (S2)
- net at U12.8 (7D): now also U11.13 (S3)
- net at U12.9 (8D): now also U11.10 (S4)
- net at U18.11 (LE), U22.11 (LE): now also J15.1 (Pin_1); no longer U13.8
- net at U28.11 (LE), U33.11 (LE): now also J15.2 (Pin_2); no longer U13.11
- net at U36.11 (LE), U39.11 (LE): now also J15.3 (Pin_3); no longer U24.3
- net at U13.5: now also J6.4 (CLK_F); no longer U30.3 (C)
- net at U30.4 (R): now also U1.8; no longer U27.11
- net at U30.7 (S): now also U1.6; no longer U27.8
- net at U27.13: now also U13.12, U13.6, U13.9, U24.1, U24.12, U24.4, U24.9
- net at U16.1 (A0): now also J7.3 (Pin_3); no longer J8.3 (Pin_3)
- net at U16.2 (A1): now also J7.2 (Pin_2); no longer J8.2 (Pin_2)
- net at U16.3 (A2): now also J7.1 (Pin_1); no longer J8.1 (Pin_1)
- net at U17.1 (A0): now also J8.3 (Pin_3); no longer J7.3 (Pin_3)
- net at U17.2 (A1): now also J8.2 (Pin_2); no longer J7.2 (Pin_2)
- net at U17.3 (A2): now also J8.1 (Pin_1); no longer J7.1 (Pin_1)
- net at U27.1: now also U27.11, J14.8 (Pin_8); no longer U6.11 (~{Y8})
- net at U13.2: now also J6.3 (CLK_R)
- net at U27.3: now also U27.10, U27.4; no longer U27.5
- new net: J15.8 (Pin_8), U60.11 (LE)
- new net: J15.9 (Pin_9), U64.11 (LE)
- new net: J10.1 (Pin_1), U7.12 (8Q)
- new net: J10.2 (Pin_2), U7.13 (7Q)
- new net: J10.3 (Pin_3), U7.14 (6Q)
- new net: J10.4 (Pin_4), U7.15 (5Q)
- new net: J10.5 (Pin_5), U7.16 (4Q)
- new net: J10.6 (Pin_6), U7.17 (3Q)
- new net: J10.7 (Pin_7), U7.18 (2Q)
- new net: J10.8 (Pin_8), U7.19 (1Q)
- new net: J10.9 (Pin_9), U12.12 (8Q)
- new net: J10.10 (Pin_10), U12.13 (7Q)
- new net: J10.11 (Pin_11), U12.14 (6Q)
- new net: J10.12 (Pin_12), U12.15 (5Q)
- new net: J10.13 (Pin_13), U12.16 (4Q)
- new net: J10.14 (Pin_14), U12.17 (3Q)
- new net: J10.15 (Pin_15), U12.18 (2Q)
- new net: J10.16 (Pin_16), U12.19 (1Q)
- new net: D1.2 (A), J14.9 (Pin_9), J6.65 (Sup), U27.2, U30.1 (Q)
- new net: U1.5, U27.8
- new net: J14.7 (Pin_7), U27.9, U68.1, U68.2
- new net: U27.12, U6.11 (~{Y8})
- new net: J14.4 (Pin_4), U24.6
- new net: J14.1 (Pin_1), U13.8
- new net: J14.2 (Pin_2), U13.11
- new net: J14.3 (Pin_3), U24.3
- new net: U27.5, U68.3
- new net: U1.10, U27.6
- new net: J14.5 (Pin_5), U24.8
- new net: J14.6 (Pin_6), U24.11
- new net: R2.2, U3.21, U3.22, U3.23, U3.24, U3.25, U3.26, U3.27, U3.28
- new net: R4.2, U3.29, U3.30, U3.31, U3.32, U3.33, U3.34, U3.35, U3.36
- new net: J4.18 (from_Bus7), U11.11 (B4), U8.9
- new net: J4.17 (from_Bus6), U11.15 (B3), U8.10
- new net: J4.16 (from_Bus5), U11.2 (B2), U8.11
- new net: J4.15 (from_Bus4), U11.6 (B1), U8.12
- new net: U11.7 (C0), U5.9 (C4)
- new net: U11.9 (C4), U19.7 (C0)
- new net: J4.11 (from_Bus0), U5.6 (B1), U8.16
- new net: J4.12 (from_Bus1), U5.2 (B2), U8.15
- new net: J4.13 (from_Bus2), U5.15 (B3), U8.14
- new net: J4.14 (from_Bus3), U5.11 (B4), U8.13
- new net: J4.19 (from_Bus8), U19.6 (B1), U8.8
- new net: J4.20 (from_Bus9), U19.2 (B2), U8.7
- new net: J4.21 (from_Bus10), U19.15 (B3), U8.6
- new net: J4.22 (from_Bus11), U19.11 (B4), U8.5
- new net: J4.23 (from_Bus12), U23.6 (B1), U8.4
- new net: J4.24 (from_Bus13), U23.2 (B2), U8.3
- new net: J4.25 (from_Bus14), U23.15 (B3), U8.2
- new net: J4.26 (from_Bus15), U23.11 (B4), U8.1
- new net: R1.2, U2.21, U2.22, U2.23, U2.24, U2.25, U2.26, U2.27, U2.28
- new net: R3.2, U2.29, U2.30, U2.31, U2.32, U2.33, U2.34, U2.35, U2.36
- new net: R5.2, U8.21, U8.22, U8.23, U8.24, U8.25, U8.26, U8.27, U8.28
- new net: R6.2, U8.29, U8.30, U8.31, U8.32, U8.33, U8.34, U8.35, U8.36
- new net: U1.3, U5.5 (A1)
- new net: D1.1 (K), R7.2
- new net: U19.9 (C4), U23.7 (C0)
- new net Dec: J5.1 (Pin_1), U1.1, U11.12 (A4), U11.14 (A3), U11.3 (A2), U11.5 (A1), U19.12 (A4), U19.14 (A3), U19.3 (A2), U19.5 (A1), U23.12 (A4), U23.14 (A3), U23.3 (A2), U23.5 (A1), U5.12 (A4), U5.14 (A3), U5.3 (A2)
- new net Inc: J5.2 (Pin_2), U1.2
Other:
- moved on the sheet: J1, J11, J12, J2, J3, J7, J8, J9, U10, U12, U13A, U13B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

Commit message: Added Siwas Register File PCB + compleateted it!
Parts:
- added J16, J17: Conn_01x01_Female, Connector_PinSocket_2.54mm:PinSocket_1x01_P2.54mm_Vertical, symbol Connector:Conn_01x01_Female
- added J18: Sup_Conn_main, Connector_PinSocket_2.54mm:PinSocket_1x03_P2.54mm_Horizontal, symbol Connector:Conn_01x03_Female
- added J19: Sup_Conn_Sec, Connector_PinSocket_2.54mm:PinSocket_1x03_P2.54mm_Horizontal, symbol Connector:Conn_01x03_Female
- J3: footprint Connector_PinHeader_2.54mm:PinHeader_1x16_P2.54mm_Vertical -> Connector_PinSocket_2.54mm:PinSocket_1x03_P2.54mm_Horizontal
- U10, U9: footprint Package_DIP:DIP-20_W7.62mm_Socket -> Package_SO:SO-20_5.3x12.6mm_P1.27mm
- U14, U15, U20, U21, U25, U26, U31, U32, U34, U35, U37, U38, U40, U41, U43, U44, U46, U47, U49, U50, U52, U53, U55, U56, U58, U59, U61, U62, U63, U65, U66, U67: footprint Package_DIP:DIP-20_W7.62mm_Socket -> Package_SO:SO-20_12.8x7.5mm_P1.27mm
Connections:
- net Const_Reg: now also J16.1 (Pin_1); no longer U16.5 (~{E1}), U29.1, U29.2
- net R_Sup: now also J19.3 (Pin_3); no longer J6.67 (Reset_Sup)
- net S_Sup: now also J19.2 (Pin_2); no longer J6.66 (Set_Sup)
- net Zero_One: now also J14.12 (Pin_12); no longer U10.2 (A1), U9.2 (A1)
- net at D1.2 (A), J14.9 (Pin_9), U27.2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: now also J19.1 (Pin_1); no longer J6.65 (Sup)
- net at J15.12 (Pin_12): now also U10.2 (A1), U9.2 (A1)
- new net: J17.1 (Pin_1), U16.5 (~{E1}), U29.1, U29.2
- new net: J18.1 (Pin_1), J6.65 (Sup)
- new net: J18.2 (Pin_2), J6.66 (Set_Sup)
- new net: J18.3 (Pin_3), J6.67 (Reset_Sup)
Other:
- moved on the sheet: J6J

Commit message: Changed Label on Register File
Parts:
- added J20, J21: Conn_01x02_Female, Connector_PinSocket_2.54mm:PinSocket_1x02_P2.54mm_Vertical, symbol Connector:Conn_01x02_Female
Connections:
- net at U13.2: now also J21.2 (Pin_2); no longer J6.3 (CLK_R)
- net at U13.5: now also J21.1 (Pin_1); no longer J6.4 (CLK_F)
- new net: J20.1 (Pin_1), J6.3 (CLK_R)
- new net: J20.2 (Pin_2), J6.4 (CLK_F)
Other:
- moved on the sheet: J6A
Changed lines of the file:
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@@
     (stroke (width 0) (type default) (color 0 0 0 0))
   )
-  (wire (pts (xy 127.635 131.445) (xy 126.365 131.445))
+  (wire (pts (xy 42.545 133.35) (xy 41.275 133.35))
     (stroke (width 0) (type default) (color 0 0 0 0))
   )
@@
     (stroke (width 0) (type default) (color 0 0 0 0))
   )
-  (wire (pts (xy 126.365 133.985) (xy 127.635 133.985))
+  (wire (pts (xy 41.275 135.89) (xy 42.545 135.89))
     (stroke (width 0) (type default) (color 0 0 0 0))
   )
@@
     (stroke (width 0) (type default) (color 0 0 0 0))
   )
-  (wire (pts (xy 126.365 139.065) (xy 174.625 139.065))
-    (stroke (width 0) (type default) (color 0 0 0 0))
-  )
   (wire (pts (xy 467.995 426.085) (xy 465.455 426.085))
     (stroke (width 0) (type default) (color 0 0 0 0))
@@
     (stroke (width 0) (type default) (color 0 0 0 0))
   )
+  (wire (pts (xy 126.365 139.065) (xy 174.625 139.065))
+    (stroke (width 0) (type default) (color 0 0 0 0))
+  )
   (wire (pts (xy 796.925 207.01) (xy 796.925 209.55))
     (stroke (width 0) (type default) (color 0 0 0 0))
@@
     (pin "1")
   )
-  (symbol (lib_id "power:+5V") (at 127.635 133.985 270) (unit 1)
+  (symbol (lib_id "power:+5V") (at 42.545 135.89 270) (unit 1)
     (in_bom yes) (on_board yes)
-    (property "Reference" "#PWR013" (id 0) (at 123.825 133.985 0)
+    (property "Reference" "#PWR013" (id 0) (at 38.735 135.89 0)
       (effects (font (size 1.27 1.27)) hide)
     )
-    (property "Value" "+5V" (id 1) (at 130.8862 134.366 90)
+    (property "Value" "+5V" (id 1) (at 45.7962 136.271 90)
       (effects (font (size 1.27 1.27)) (justify left))
     )
-    (property "Footprint" "" (id 2) (at 127.635 133.985 0)
+    (property "Footprint" "" (id 2) (at 42.545 135.89 0)
       (effects (font (size 1.27 1.27)) hide)
     )
-    (property "Datasheet" "" (id 3) (at 127.635 133.985 0)
+    (property "Datasheet" "" (id 3) (at 42.545 135.89 0)
       (effects (font (size 1.27 1.27)) hide)
     )
     (pin "1")
   )
-  (symbol (lib_id "power:GND") (at 127.635 131.445 90) (unit 1)
+  (symbol (lib_id "power:GND") (at 42.545 133.35 90) (unit 1)
     (in_bom yes) (on_board yes)
-    (property "Reference" "#PWR012" (id 0) (at 133.985 131.445 0)
+    (property "Reference" "#PWR012" (id 0) (at 48.895 133.35 0)
       (effects (font (size 1.27 1.27)) hide)
     )
-    (property "Value" "GND" (id 1) (at 130.8862 131.318 90)
+    (property "Value" "GND" (id 1) (at 45.7962 133.223 90)
       (effects (font (size 1.27 1.27)) (justify right))
     )
-    (property "Footprint" "" (id 2) (at 127.635 131.445 0)
+    (property "Footprint" "" (id 2) (at 42.545 133.35 0)
       (effects (font (size 1.27 1.27)) hide)
     )
-    (property "Datasheet" "" (id 3) (at 127.635 131.445 0)
+    (property "Datasheet" "" (id 3) (at 42.545 133.35 0)
       (effects (font (size 1.27 1.27)) hide)
     )
@@
     (pin "2")
   )
+  (symbol (lib_id "Connector:Conn_01x02_Female") (at 46.355 138.43 0) (unit 1)
+    (in_bom yes) (on_board yes)
+    (property "Reference" "J20" (id 0) (at 45.085 145.415 0)
+      (effects (font (size 1.27 1.27)) (justify left))
+    )
+    (property "Value" "Conn_01x02_Female" (id 1) (at 39.37 142.875 0)
+      (effects (font (size 1.27 1.27)) (justify left))
+    )
+    (property "Footprint" "Connector_PinSocket_2.54mm:PinSocket_1x02_P2.54mm_Vertical" (id 2) (at 46.355 138.43 0)
+      (effects (font (size 1.27 1.27)) hide)
+    )
+    (property "Datasheet" "~" (id 3) (at 46.355 138.43 0)
+      (effects (font (size 1.27 1.27)) hide)
+    )
+    (pin "1")
+    (pin "2")
+  )
   (symbol (lib_id "power:PWR_FLAG") (at 57.15 364.49 0) (unit 1)
     (in_bom yes) (on_board yes) (fields_autoplaced)
@@
     (pin "1")
   )
-  (symbol (lib_id "Computer_Component_Library:Bus_Connector") (at 122.555 135.255 0) (unit 1)
+  (symbol (lib_id "Computer_Component_Library:Bus_Connector") (at 37.465 137.16 0) (unit 1)
     (in_bom yes) (on_board yes)
-    (property "Reference" "J6" (id 0) (at 107.315 134.62 0))
-    (property "Value" "Bus_Connector" (id 1) (at 107.315 136.525 0))
-    (property "Footprint" "Computer_Component_Library:PinHeader_1x78_P2.54mm_Horizontal" (id 2) (at 89.535 151.765 0)
+    (property "Reference" "J6" (id 0) (at 22.225 136.525 0))
+    (property "Value" "Bus_Connector" (id 1) (at 22.225 138.43 0))
+    (property "Footprint" "Computer_Component_Library:PinHeader_1x78_P2.54mm_Horizontal" (id 2) (at 4.445 153.67 0)
       (effects (font (size 1.27 1.27)) hide)
     )
-    (property "Datasheet" "" (id 3) (at 89.535 151.765 0)
+    (property "Datasheet" "" (id 3) (at 4.445 153.67 0)
       (effects (font (size 1.27 1.27)) hide)
     )
@@
     (pin "1")
   )
+  (symbol (lib_id "Connector:Conn_01x02_Female") (at 121.285 139.065 180) (unit 1)
+    (in_bom yes) (on_board yes)
+    (property "Reference" "J21" (id 0) (at 120.015 136.525 0)
+      (effects (font (size 1.27 1.27)) (justify left))
+    )
+    (property "Value" "Conn_01x02_Female" (id 1) (at 120.65 139.065 0)
+      (effects (font (size 1.27 1.27)) (justify left))
+    )
+    (property "Footprint" "Connector_PinSocket_2.54mm:PinSocket_1x02_P2.54mm_Vertical" (id 2) (at 121.285 139.065 0)
+      (effects (font (size 1.27 1.27)) hide)
+    )
+    (property "Datasheet" "~" (id 3) (at 121.285 139.065 0)
+      (effects (font (size 1.27 1.27)) hide)
+    )
+    (pin "1")
+    (pin "2")
+  )
   (symbol (lib_id "power:PWR_FLAG") (at 33.02 499.745 180) (unit 1)
     (in_bom yes) (on_board yes) (fields_autoplaced)
@@
       (reference "J19") (unit 1) (value "Sup_Conn_Sec") (footprint "Connector_PinSocket_2.54mm:PinSocket_1x03_P2.54mm_Horizontal")
     )
+    (path "/708514ad-846a-48ab-9091-bea41c0f2b85"
+      (reference "J20") (unit 1) (value "Conn_01x02_Female") (footprint "Connector_PinSocket_2.54mm:PinSocket_1x02_P2.54mm_Vertical")
+    )
+    (path "/bc44eac0-510e-46a9-9a4d-eb26bb53186f"
+      (reference "J21") (unit 1) (value "Conn_01x02_Female") (footprint "Connector_PinSocket_2.54mm:PinSocket_1x02_P2.54mm_Vertical")
+    )
     (path "/e88839e7-bce2-4e2a-9e44-2ebe779718f6"
