File: circets/Activation_Module/Activation_Module/Activation_Module.sch (KiCad schematic (older format))
At the start: 50 parts, among them J1 Bus_Connector, J2 To_Bus, J3 From_Bus, J4 Mode_R, J5 Mode_W, J6 Enable Connector, SW1 SW_DIP_x04, SW2 SW_DIP_x04, U1 74HC541, U10 74HC541, U11 74HC00, U12 74HC541, U13 74HC541, U14 74HC541, U15 74LS86, U16 74LS86, U17 74LS32, U18 74LS32, U19 74157, U2 74HC541, U20 74157, U3 74LS86, U4 74LS86, U5 74LS32, U6 74LS32, U7 74HC541, U8 74HC541, U9 74HC00

Commit message: Fixed Issue with wrong pins in activation Module!
Parts:
- removed unit 5 of J1
- removed unit 7 of J1
- added J? (x2): Bus_Connector, symbol Computer_Component_Library:Bus_Connector
- J1: symbol Computer_Component_Library:Bus_Connector -> Activation_Module-rescue:Bus_Connector-Computer_Component_Library
Connections:
- net at U4.2: now also J?.47 (WE2:3)
- net at U4.5: now also J?.48 (WE2:4)
- net at U4.10: now also J?.49 (WE2:5)
- net at U4.13: now also J?.50 (WE2:6)
- net at U16.2: now also J?.61 (RE2:3)
- net at U16.5: now also J?.62 (RE2:4)
- net at U16.10: now also J?.63 (RE2:5)
- net at U16.13: now also J?.64 (RE2:6)
- net at U19.13 (I1c): now also J?.60 (RE2:2)
- net at U19.14 (I0c): now also J?.46 (WE2:2)
- net at U19.2 (I0a): now also J?.44 (WE2:0)
- net at U19.3 (I1a): now also J?.58 (RE2:0)
- net at U19.5 (I0b): now also J?.45 (WE2:1)
- net at U19.6 (I1b): now also J?.59 (RE2:1)
Changed lines of the file:
@@
 	4700 10500 4700 9650
 $Comp
-L Computer_Component_Library:Bus_Connector J1
+L Activation_Module-rescue:Bus_Connector-Computer_Component_Library J1
 U 2 1 62E54F07
 P 4750 10650
@@
 $EndComp
 $Comp
-L Computer_Component_Library:Bus_Connector J1
+L Activation_Module-rescue:Bus_Connector-Computer_Component_Library J1
 U 3 1 62E59683
 P 10000 10650
@@
 	2700 4850 600  4850
 $Comp
-L Computer_Component_Library:Bus_Connector J1
+L Activation_Module-rescue:Bus_Connector-Computer_Component_Library J1
 U 4 1 63F6778F
 P 1750 1000
@@
 $EndComp
 $Comp
-L Computer_Component_Library:Bus_Connector J1
-U 5 1 63F6A1B9
-P 900 1000
-F 0 "J1" V 500 950 50  0000 L CNN
-F 1 "Bus_Connector" V 600 900 50  0000 L CNN
-F 2 "Computer_Component_Library:BusConnector" H -400 350 50  0001 C CNN
-F 3 "" H -400 350 50  0001 C CNN
-	5    900  1000
-	0    1    1    0
-$EndComp
-$Comp
-L Computer_Component_Library:Bus_Connector J1
+L Activation_Module-rescue:Bus_Connector-Computer_Component_Library J1
 U 6 1 63F6D143
 P 9750 1000
@@
 F 3 "" H 8450 350 50  0001 C CNN
 	6    9750 1000
-	0    1    1    0
-$EndComp
-$Comp
-L Computer_Component_Library:Bus_Connector J1
-U 7 1 63F6FE35
-P 8850 1000
-F 0 "J1" V 8450 950 50  0000 L CNN
-F 1 "Bus_Connector" V 8550 900 50  0000 L CNN
-F 2 "Computer_Component_Library:BusConnector" H 7550 350 50  0001 C CNN
-F 3 "" H 7550 350 50  0001 C CNN
-	7    8850 1000
 	0    1    1    0
 $EndComp
@@
 	6500 5100 6500 5050
 $Comp
-L Computer_Component_Library:Bus_Connector J1
+L Activation_Module-rescue:Bus_Connector-Computer_Component_Library J1
 U 1 1 6DC16388
 P 6700 5250
@@
 Wire Wire Line
 	5850 2200 5850 2150
+$Comp
+L Computer_Component_Library:Bus_Connector J?
+U 5 1 61D797A8
+P 900 1000
+F 0 "J?" V 726 1388 50  0000 L CNN
+F 1 "Bus_Connector" V 817 1388 50  0000 L CNN
+F 2 "" H -400 350 50  0001 C CNN
+F 3 "" H -400 350 50  0001 C CNN
+	5    900  1000
+	0    1    1    0
+$EndComp
+$Comp
+L Computer_Component_Library:Bus_Connector J?
+U 7 1 61D96A01
+P 8850 1000
+F 0 "J?" V 8450 950 50  0000 L CNN
+F 1 "Bus_Connector" V 8550 900 50  0000 L CNN
+F 2 "" H 7550 350 50  0001 C CNN
+F 3 "" H 7550 350 50  0001 C CNN
+	7    8850 1000
+	0    1    1    0
+$EndComp
 $EndSCHEMATC

Commit message: Added correct connectors to AM
Parts:
- removed J2: To_Bus, Connector_PinHeader_2.54mm:PinHeader_1x16_P2.54mm_Vertical, symbol Connector:Conn_01x16_Female
- removed J3: From_Bus, Connector_PinHeader_2.54mm:PinHeader_1x16_P2.54mm_Vertical, symbol Connector:Conn_01x16_Female
- removed J4: Mode_R, Connector_PinSocket_2.54mm:PinSocket_1x03_P2.54mm_Vertical, symbol Connector:Conn_01x03_Female
- removed J5: Mode_W, Connector_PinSocket_2.54mm:PinSocket_1x03_P2.54mm_Vertical, symbol Connector:Conn_01x03_Female
- removed J6: Enable Connector, Connector_PinSocket_2.54mm:PinSocket_1x03_P2.54mm_Vertical, symbol Connector:Conn_01x03_Female
- added U? (x5): AM-Connector, symbol Computer_Component_Library:AM-Connector
Connections:
- net RE: now also U?.10 (RE), U?.7 (WE_R)
- net WE_F: now also U?.9 (WE)
- net WE_R: now also U?.8 (WE_F)
- net at U14.11 (Y8), U8.11 (Y8): now also U?.26 (from_Bus15)
- net at U14.12 (Y7), U8.12 (Y7): now also U?.25 (from_Bus14)
- net at U14.13 (Y6), U8.13 (Y6): now also U?.24 (from_Bus13)
- net at U14.14 (Y5), U8.14 (Y5): now also U?.23 (from_Bus12)
- net at U14.15 (Y4), U8.15 (Y4): now also U?.22 (from_Bus11)
- net at U14.16 (Y3), U8.16 (Y3): now also U?.21 (from_Bus10)
- net at U14.17 (Y2), U8.17 (Y2): now also U?.20 (from_Bus9)
- net at U14.18 (Y1), U8.18 (Y1): now also U?.19 (from_Bus8)
- net at U13.11 (Y8), U7.11 (Y8): now also U?.18 (from_Bus7)
- net at U13.12 (Y7), U7.12 (Y7): now also U?.17 (from_Bus6)
- net at U13.13 (Y6), U7.13 (Y6): now also U?.16 (from_Bus5)
- net at U13.14 (Y5), U7.14 (Y5): now also U?.15 (from_Bus4)
- net at U13.15 (Y4), U7.15 (Y4): now also U?.14 (from_Bus3)
- net at U13.16 (Y3), U7.16 (Y3): now also U?.13 (from_Bus2)
- net at U13.17 (Y2), U7.17 (Y2): now also U?.12 (from_Bus1)
- net at U13.18 (Y1), U7.18 (Y1): now also U?.11 (from_Bus0)
- net at U1.2 (A1), U10.2 (A1): now also U?.42 (to_Bus15)
- net at U12.3 (A2), U2.3 (A2): now also U?.33 (to_Bus6)
- net at U12.4 (A3), U2.4 (A3): now also U?.32 (to_Bus5)
- net at U12.5 (A4), U2.5 (A4): now also U?.31 (to_Bus4)
- net at U12.6 (A5), U2.6 (A5): now also U?.30 (to_Bus3)
- net at U12.7 (A6), U2.7 (A6): now also U?.29 (to_Bus2)
- net at U12.8 (A7), U2.8 (A7): now also U?.28 (to_Bus1)
- net at U12.9 (A8), U2.9 (A8): now also U?.27 (to_Bus0)
- net at U1.3 (A2), U10.3 (A2): now also U?.41 (to_Bus14)
- net at U1.4 (A3), U10.4 (A3): now also U?.40 (to_Bus13)
- net at U1.5 (A4), U10.5 (A4): now also U?.39 (to_Bus12)
- net at U1.6 (A5), U10.6 (A5): now also U?.38 (to_Bus11)
- net at U1.7 (A6), U10.7 (A6): now also U?.37 (to_Bus10)
- net at U1.8 (A7), U10.8 (A7): now also U?.36 (to_Bus9)
- net at U1.9 (A8), U10.9 (A8): now also U?.35 (to_Bus8)
- net at U12.2 (A1), U2.2 (A1): now also U?.34 (to_Bus7)
- net at U19.12 (Qc): now also U?.3 (Mode_R2)
- net at U19.4 (Qa): now also U?.1 (Mode_R0)
- net at U19.7 (Qb): now also U?.2 (Mode_R1)
- net at U20.12 (Qc): now also U?.6 (Mode_W2)
- net at U20.4 (Qa): now also U?.4 (Mode_W0)
- net at U20.7 (Qb): now also U?.5 (Mode_W1)
Changed lines of the file:
@@
 Sheet 1 1
 Title "Activation Module"
-Date "2021-12-21"
-Rev "v0.3"
+Date "2022-01-05"
+Rev "v0.4"
 Comp ""
 Comment1 ""
@@
 	3500 6400 3500 6850
 Wire Wire Line
-	900  8450 900  6400
+	900  8450 900  7050
 Connection ~ 900  8450
 Wire Wire Line
-	1000 8400 1000 6400
+	1000 8400 1000 7050
 Connection ~ 1000 8400
 Wire Wire Line
-	1100 8350 1100 6400
+	1100 8350 1100 7050
 Connection ~ 1100 8350
 Wire Wire Line
-	1200 6400 1200 8300
+	1200 7050 1200 8300
 Connection ~ 1200 8300
 Wire Wire Line
-	1300 8250 1300 6400
+	1300 8250 1300 7050
 Connection ~ 1300 8250
 Wire Wire Line
-	1400 6400 1400 8200
+	1400 7050 1400 8200
 Connection ~ 1400 8200
 Wire Wire Line
-	1500 8150 1500 6400
+	1500 8150 1500 7050
 Connection ~ 1500 8150
 Wire Wire Line
-	1600 6400 1600 8100
+	1600 7050 1600 8100
 Connection ~ 1600 8100
 Wire Wire Line
-	1700 6400 1700 8050
+	1700 7050 1700 8050
 Wire Wire Line
 	1700 8050 2200 8050
@@
 	2300 8000 1800 8000
 Wire Wire Line
-	1800 8000 1800 6400
+	1800 8000 1800 7050
 Connection ~ 2300 8000
 Wire Wire Line
-	1900 6400 1900 7950
+	1900 7050 1900 7950
 Wire Wire Line
 	1900 7950 2400 7950
@@
 	2500 7900 2000 7900
 Wire Wire Line
-	2000 7900 2000 6400
+	2000 7900 2000 7050
 Connection ~ 2500 7900
 Wire Wire Line
-	2100 6400 2100 7850
+	2100 7050 2100 7850
 Wire Wire Line
 	2100 7850 2600 7850
@@
 	2700 7800 2200 7800
 Wire Wire Line
-	2200 7800 2200 6400
+	2200 7800 2200 7050
 Connection ~ 2700 7800
 Wire Wire Line
-	2300 6400 2300 7750
+	2300 7050 2300 7750
 Wire Wire Line
 	2300 7750 2800 7750
@@
 	2900 7700 2400 7700
 Wire Wire Line
-	2400 7700 2400 6400
+	2400 7700 2400 7050
 Connection ~ 2900 7700
-$Comp
-L Connector:Conn_01x16_Female J2
-U 1 1 62D9B096
-P 1600 6200
-F 0 "J2" V 1550 5300 50  0000 C CNN
-F 1 "To_Bus" V 1450 5250 50  0000 C CNN
-F 2 "Connector_PinHeader_2.54mm:PinHeader_1x16_P2.54mm_Vertical" H 1600 6200 50  0001 C CNN
-F 3 "~" H 1600 6200 50  0001 C CNN
-	1    1600 6200
-	0    -1   -1   0
-$EndComp
-$Comp
-L Connector:Conn_01x16_Female J3
-U 1 1 62DA0E02
-P 4200 6200
-F 0 "J3" V 4150 5300 50  0000 C CNN
-F 1 "From_Bus" V 4050 5200 50  0000 C CNN
-F 2 "Connector_PinHeader_2.54mm:PinHeader_1x16_P2.54mm_Vertical" H 4200 6200 50  0001 C CNN
-F 3 "~" H 4200 6200 50  0001 C CNN
-	1    4200 6200
-	0    -1   -1   0
-$EndComp
 $Comp
 L 74xx:74LS32 U6
@@
 Wire Wire Line
 	6000 4250 6350 4250
-$Comp
-L Connector:Conn_01x03_Female J6
-U 1 1 6ED25AAF
-P 8100 3750
-F 0 "J6" V 8250 4200 50  0000 R CNN
-F 1 "Enable Connector" V 8150 4200 50  0000 R CNN
-F 2 "Connector_PinSocket_2.54mm:PinSocket_1x03_P2.54mm_Vertical" H 8100 3750 50  0001 C CNN
-F 3 "~" H 8100 3750 50  0001 C CNN
-	1    8100 3750
-	0    -1   -1   0
-$EndComp
 Wire Wire Line
 	8000 3950 8000 4150
@@
 Wire Wire Line
 	6000 5400 6550 5400
-$Comp
-L Connector:Conn_01x03_Female J4
-U 1 1 6F517F4D
-P 13300 6750
-F 0 "J4" V 13450 6600 50  0000 L CNN
-F 1 "Mode_R" V 13350 6600 50  0000 L CNN
-F 2 "Connector_PinSocket_2.54mm:PinSocket_1x03_P2.54mm_Vertical" H 13300 6750 50  0001 C CNN
-F 3 "~" H 13300 6750 50  0001 C CNN
-	1    13300 6750
-	0    -1   -1   0
-$EndComp
-$Comp
-L Connector:Conn_01x03_Female J5
-U 1 1 6F578562
-P 15450 6750
-F 0 "J5" V 15600 6600 50  0000 L CNN
-F 1 "Mode_W" V 15500 6600 50  0000 L CNN
-F 2 "Connector_PinSocket_2.54mm:PinSocket_1x03_P2.54mm_Vertical" H 15450 6750 50  0001 C CNN
-F 3 "~" H 15450 6750 50  0001 C CNN
-	1    15450 6750
-	0    -1   -1   0
-$EndComp
 Text Notes 15100 6450 0    118  ~ 0
 Mode-Router
@@
 	13150 7000 13200 7000
 Wire Wire Line
-	13200 7000 13200 6950
-Wire Wire Line
-	13300 6950 13300 7200
-Wire Wire Line
 	13300 7200 13150 7200
 Wire Wire Line
 	13150 7400 13400 7400
 Wire Wire Line
-	13400 7400 13400 6950
-Wire Wire Line
-	15350 6950 15350 7000
-Wire Wire Line
 	15350 7000 15300 7000
 Wire Wire Line
-	15450 6950 15450 7200
-Wire Wire Line
 	15450 7200 15300 7200
-Wire Wire Line
-	15550 6950 15550 7400
 Wire Wire Line
 	15550 7400 15300 7400
@@
 	0    1    1    0
 $EndComp
+$Comp
+L Computer_Component_Library:AM-Connector U?
+U 1 1 62917F1A
+P 13450 8250
+F 0 "U?" V 13283 7922 50  0000 R CNN
+F 1 "AM-Connector" V 13192 7922 50  0000 R CNN
+F 2 "" H 13600 8250 50  0001 C CNN
+F 3 "" H 13600 8250 50  0001 C CNN
+	1    13450 8250
+	0    -1   -1   0
+$EndComp
+Wire Wire Line
+	13200 7000 13200 8100
+Wire Wire Line
+	13300 7200 13300 8100
+Wire Wire Line
+	13400 7400 13400 8100
+Wire Wire Line
+	15350 7000 15350 7800
+Wire Wire Line
+	15350 7800 13500 7800
+Wire Wire Line
+	13500 7800 13500 8100
+Wire Wire Line
+	13600 8100 13600 7850
+Wire Wire Line
+	13600 7850 15450 7850
+Wire Wire Line
+	15450 7850 15450 7200
+Wire Wire Line
+	15550 7400 15550 7900
+Wire Wire Line
+	15550 7900 13700 7900
+Wire Wire Line
+	13700 7900 13700 8100
+$Comp
+L Computer_Component_Library:AM-Connector U?
+U 2 1 62D6A39E
+P 8100 3800
+F 0 "U?" V 7963 3988 50  0000 L CNN
+F 1 "AM-Connector" V 8054 3988 50  0000 L CNN
+F 2 "" H 8250 3800 50  0001 C CNN
+F 3 "" H 8250 3800 50  0001 C CNN
+	2    8100 3800
+	0    1    1    0
+$EndComp
+$Comp
+L Computer_Component_Library:AM-Connector U?
+U 3 1 62D8CC7E
+P 14500 3000
+F 0 "U?" V 14390 3088 50  0000 L CNN
+F 1 "AM-Connector" V 14481 3088 50  0000 L CNN
+F 2 "" H 14650 3000 50  0001 C CNN
+F 3 "" H 14650 3000 50  0001 C CNN
+	3    14500 3000
+	0    1    1    0
+$EndComp
+Wire Wire Line
+	14500 3150 14500 3200
+Connection ~ 14500 3200
+$Comp
+L Computer_Component_Library:AM-Connector U?
+U 4 1 62E93C1C
+P 4250 6250
+F 0 "U?" V 3877 5422 50  0000 R CNN
+F 1 "AM-Connector" V 3968 5422 50  0000 R CNN
+F 2 "" H 4400 6250 50  0001 C CNN
+F 3 "" H 4400 6250 50  0001 C CNN
+	4    4250 6250
+	0    -1   1    0
+$EndComp
+$Comp
+L Computer_Component_Library:AM-Connector U?
+U 5 1 62E9F6AB
+P 1650 6900
+F 0 "U?" V 1326 7738 50  0000 L CNN
+F 1 "AM-Connector" V 1417 7738 50  0000 L CNN
+F 2 "" H 1800 6900 50  0001 C CNN
+F 3 "" H 1800 6900 50  0001 C CNN
+	5    1650 6900
+	0    1    1    0
+$EndComp

Commit message: Started Creating Activation Module PCB
Parts:
- removed J1: Bus_Connector, Computer_Component_Library:BusConnector, symbol Activation_Module-rescue:Bus_Connector-Computer_Component_Library
- removed J? (x2): Bus_Connector, symbol Computer_Component_Library:Bus_Connector
- removed unit 2 of U11
- removed unit 4 of U11
- removed unit 4 of U17
- removed unit 4 of U6
- removed U9: 74HC00, Package_DIP:DIP-14_W7.62mm_Socket, symbol 74xx:74HC00
- added C7, C8: 0.1µF, Capacitor_THT:C_Disc_D6.0mm_W2.5mm_P5.00mm, symbol Device:C
- added J1: Bus_Connector, Computer_Component_Library:PinSocket_1x78_P2.00mm_Horizontal, symbol Computer_Component_Library:Bus_Connector
- added J2: Conn_01x03_Male, Connector_PinSocket_2.00mm:PinSocket_1x03_P2.00mm_Vertical, symbol Connector:Conn_01x03_Male
- added U19: 74LS08, Package_DIP:DIP-14_W7.62mm_Socket, symbol 74xx:74LS08
- added U22: 74LS32, Package_DIP:DIP-14_W7.62mm_Socket, symbol 74xx:74LS32
- added U23: 74LS00, Package_DIP:DIP-14_W7.62mm_Socket, symbol 74xx:74LS00
- U1, U10: footprint Computer_Component_Library:74HC541-PDIP -> Package_DIP:DIP-20_W7.62mm_Socket
- U11: renamed from U12; footprint Computer_Component_Library:74HC541-PDIP -> Package_DIP:DIP-20_W7.62mm_Socket
- U14: renamed from U13; footprint Computer_Component_Library:74HC541-PDIP -> Package_DIP:DIP-20_W7.62mm_Socket
- U17: renamed from U14; footprint Computer_Component_Library:74HC541-PDIP -> Package_DIP:DIP-20_W7.62mm_Socket
- U2: renamed from U?; footprint (none) -> Computer_Component_Library:PinSocket_1x42_P2.00mm_Horizontal
- U3: renamed from U2; footprint Computer_Component_Library:74HC541-PDIP -> Package_DIP:DIP-20_W7.62mm_Socket
- U8: renamed from U7; footprint Computer_Component_Library:74HC541-PDIP -> Package_DIP:DIP-20_W7.62mm_Socket
- U9: renamed from U8; footprint Computer_Component_Library:74HC541-PDIP -> Package_DIP:DIP-20_W7.62mm_Socket
- renumbered R8 to R10, R9 to R5, R10 to R6, R5 to R7, R6 to R8, R7 to R9, U15 to U12, U16 to U13, U18 to U15, U17 to U15, U17 to U16, U18 to U16, U11 to U18, U19 to U20, U20 to U21, U3 to U4, U4 to U5, U5 to U6, U18 to U7, U6 to U7, U5 to U7
Connections:
- net +5V: now also C7.2, C8.2, J1.2 (Vcc), U19.7 (GND), U22.7 (GND)
- net GND: now also C7.1, C8.1, J1.1 (GND), J2.3 (Pin_3), U19.14 (VCC), U22.14 (VCC)
- net WE_F: now also U2.8 (WE_F), U19.3; no longer U2.9 (WE)
- net WE_R: now also U2.7 (WE_R), U19.6; no longer U2.8 (WE_F)
- net WE1:3: now reaches U4.2
- net WE1:3: now also J1.40 (WE1:3)
- net WE1:4: now reaches U4.5
- net WE1:4: now also J1.41 (WE1:4)
- net WE1:5: now reaches U4.10
- net WE1:5: now also J1.42 (WE1:5)
- net at U4.8: now also U7.9; no longer U7.5
- net WE1:6: now reaches U4.13
- net WE1:6: now also J1.43 (WE1:6)
- net WE2:3: now reaches U5.2
- net WE2:3: now also J1.47 (WE2:3)
- net WE2:4: now reaches U5.5
- net WE2:4: now also J1.48 (WE2:4)
- net WE2:5: now reaches U5.10
- net WE2:5: now also J1.49 (WE2:5)
- net WE2:6: now reaches U5.13
- net WE2:6: now also J1.50 (WE2:6)
- net RE1:3: now reaches U12.2
- net RE1:3: now also J1.54 (RE1:3)
- net RE1:4: now reaches U12.5
- net RE1:4: now also J1.55 (RE1:4)
- net RE1:5: now reaches U12.10
- net RE1:5: now also J1.56 (RE1:5)
- net at U12.8: now also U16.9; no longer U16.5
- net RE1:6: now reaches U12.13
- net RE1:6: now also J1.57 (RE1:6)
- net RE2:3: now reaches U13.2
- net RE2:3: now also J1.61 (RE2:3)
- net RE2:4: now reaches U13.5
- net RE2:4: now also J1.62 (RE2:4)
- net RE2:5: now reaches U13.10
- net RE2:5: now also J1.63 (RE2:5)
- net RE2:6: now reaches U13.13
- net RE2:6: now also J1.64 (RE2:6)
- net at U18.3: now also U2.9 (WE), U19.1, U19.4
- net at U16.6: now also U22.12; no longer U16.9
- net ~RE1: now reaches D3.1 (K), U1.1 (~G1), U20.1 (A/B), U3.1 (~G1), U7.12
- net ~RE1: now also U22.11; no longer U16.8
- net ~RE2: now reaches D4.1 (K), U10.1 (~G1), U11.1 (~G1), U7.13
- net ~RE2: now also U22.8; no longer U15.8
- net RE1:0: now reaches U20.2 (I0a)
- net RE1:0: now also J1.51 (RE1:0)
- net RE1:1: now reaches U20.5 (I0b)
- net RE1:1: now also J1.52 (RE1:1)
- net RE1:2: now reaches U20.14 (I0c)
- net RE1:2: now also J1.53 (RE1:2)
- net RE2:0: now reaches U20.3 (I1a)
- net RE2:0: now also J1.58 (RE2:0)
- net RE2:1: now reaches U20.6 (I1b)
- net RE2:1: now also J1.59 (RE2:1)
- net RE2:2: now reaches U20.13 (I1c)
- net RE2:2: now also J1.60 (RE2:2)
- net at U18.10: now also U18.9, U7.11
- net at U18.8: now also U2.10 (RE)
- net at U7.6: now also U22.4; no longer U7.9
- net ~WE1: now reaches D1.1 (K), U21.1 (A/B), U6.12, U8.19 (~G2), U9.19 (~G2)
- net ~WE1: now also U22.6; no longer U7.8
- net ~WE2: now reaches D2.1 (K), U14.19 (~G2), U17.19 (~G2), U6.13
- net ~WE2: now also U22.3; no longer U6.8
- net at U3.18 (Y1), U9.2 (A1): now also J1.13 (BUS1:8)
- net at U3.17 (Y2), U9.3 (A2): now also J1.14 (BUS1:9)
- net at U3.16 (Y3), U9.4 (A3): now also J1.15 (BUS1:A)
- net at U3.15 (Y4), U9.5 (A4): now also J1.16 (BUS1:B)
- net at U3.14 (Y5), U9.6 (A5): now also J1.17 (BUS1:C)
- net at U3.13 (Y6), U9.7 (A6): now also J1.18 (BUS1:D)
- net at U3.12 (Y7), U9.8 (A7): now also J1.19 (BUS1:E)
- net at U3.11 (Y8), U9.9 (A8): now also J1.20 (BUS1:F)
- net at U1.18 (Y1), U8.2 (A1): now also J1.5 (BUS1:0)
- net at U1.17 (Y2), U8.3 (A2): now also J1.6 (BUS1:1)
- net at U1.16 (Y3), U8.4 (A3): now also J1.7 (BUS1:2)
- net at U1.15 (Y4), U8.5 (A4): now also J1.8 (BUS1:3)
- net at U1.14 (Y5), U8.6 (A5): now also J1.9 (BUS1:4)
- net at U1.13 (Y6), U8.7 (A6): now also J1.10 (BUS1:5)
- net at U1.12 (Y7), U8.8 (A7): now also J1.11 (BUS1:6)
- net at U1.11 (Y8), U8.9 (A8): now also J1.12 (BUS1:7)
- net at U10.18 (Y1), U14.2 (A1): now also J1.21 (BUS2:0)
- net at U10.17 (Y2), U14.3 (A2): now also J1.22 (BUS2:1)
- net at U10.16 (Y3), U14.4 (A3): now also J1.23 (BUS2:2)
- net at U10.15 (Y4), U14.5 (A4): now also J1.24 (BUS2:3)
- net at U10.14 (Y5), U14.6 (A5): now also J1.25 (BUS2:4)
- net at U10.13 (Y6), U14.7 (A6): now also J1.26 (BUS2:5)
- net at U10.12 (Y7), U14.8 (A7): now also J1.27 (BUS2:6)
- net at U10.11 (Y8), U14.9 (A8): now also J1.28 (BUS2:7)
- net at U17.2 (A1): now also U11.18 (Y1), J1.29 (BUS2:8)
- net at U11.17 (Y2), U17.3 (A2): now also J1.30 (BUS2:9)
- net at U11.16 (Y3), U17.4 (A3): now also J1.31 (BUS2:A)
- net at U11.15 (Y4), U17.5 (A4): now also J1.32 (BUS2:B)
- net at U11.14 (Y5), U17.6 (A5): now also J1.33 (BUS2:C)
- net at U11.13 (Y6), U17.7 (A6): now also J1.34 (BUS2:D)
- net at U11.12 (Y7), U17.8 (A7): now also J1.35 (BUS2:E)
- net at U11.11 (Y8), U17.9 (A8): now also J1.36 (BUS2:F)
- net at U11.9 (A8), U3.9 (A8): now also U2.42 (to_Bus15); no longer U2.27 (to_Bus0)
- net at U11.8 (A7), U3.8 (A7): now also U2.41 (to_Bus14); no longer U2.28 (to_Bus1)
- net at U11.7 (A6), U3.7 (A6): now also U2.40 (to_Bus13); no longer U2.29 (to_Bus2)
- net at U11.6 (A5), U3.6 (A5): now also U2.39 (to_Bus12); no longer U2.30 (to_Bus3)
- net at U11.5 (A4), U3.5 (A4): now also U2.38 (to_Bus11); no longer U2.31 (to_Bus4)
- net at U11.4 (A3), U3.4 (A3): now also U2.37 (to_Bus10); no longer U2.32 (to_Bus5)
- net at U11.3 (A2), U3.3 (A2): now also U2.36 (to_Bus9); no longer U2.33 (to_Bus6)
- net at U11.2 (A1), U3.2 (A1): now also U2.35 (to_Bus8); no longer U2.34 (to_Bus7)
- net at U1.9 (A8), U10.9 (A8): now also U2.34 (to_Bus7); no longer U2.35 (to_Bus8)
- net at U1.8 (A7), U10.8 (A7): now also U2.33 (to_Bus6); no longer U2.36 (to_Bus9)
- net at U1.7 (A6), U10.7 (A6): now also U2.32 (to_Bus5); no longer U2.37 (to_Bus10)
- net at U1.6 (A5), U10.6 (A5): now also U2.31 (to_Bus4); no longer U2.38 (to_Bus11)
- net at U1.5 (A4), U10.5 (A4): now also U2.30 (to_Bus3); no longer U2.39 (to_Bus12)
- net at U1.4 (A3), U10.4 (A3): now also U2.29 (to_Bus2); no longer U2.40 (to_Bus13)
- net at U1.3 (A2), U10.3 (A2): now also U2.28 (to_Bus1); no longer U2.41 (to_Bus14)
- net at U1.2 (A1), U10.2 (A1): now also U2.27 (to_Bus0); no longer U2.42 (to_Bus15)
- net WE2:2: now reaches U21.13 (I1c)
- net WE2:2: now also J1.46 (WE2:2)
- net WE1:2: now reaches U21.14 (I0c)
- net WE1:2: now also J1.39 (WE1:2)
- net WE1:0: now reaches U21.2 (I0a)
- net WE1:0: now also J1.37 (WE1:0)
- net WE2:0: now reaches U21.3 (I1a)
- net WE2:0: now also J1.44 (WE2:0)
- net WE1:1: now reaches U21.5 (I0b)
- net WE1:1: now also J1.38 (WE1:1)
- net WE2:1: now reaches U21.6 (I1b)
- net WE2:1: now also J1.45 (WE2:1)
- removed net RE: U2.10 (RE), U2.7 (WE_R), U7.11
- new net: U16.5, U16.8
- new net: U15.8, U22.9
- new net: J2.1 (Pin_1), U23.6
- new net: J1.65 (Sup), U23.4, U23.5
- new net: U22.1, U6.8
- new net: U7.5, U7.8
- new net: J1.4 (CLK_F), U19.2
- new net: J1.3 (CLK_R), U19.5
- new net ~SUP: J2.2 (Pin_2), U22.10, U22.13, U22.2, U22.5
Other:
- moved on the sheet: C3, C4, D1, D2, D3, D4, R10, R11, R12, R5, R6, R7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
