File: circets/Activation_Module/Activation_Module/Activation_Module.kicad_sch (KiCad schematic)
At the start: 51 parts, among them J1 Bus_Connector, J2 Conn_01x03_Male, SW1 SW_DIP_x04, SW2 SW_DIP_x04, U1 74HC541, U10 74HC541, U11 74HC541, U12 74LS86, U13 74LS86, U14 74HC541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

Commit message: RedesignedPCB Layout for Activation Module
Parts:
- removed U23: 74LS00, Package_DIP:DIP-14_W7.62mm_Socket, symbol 74xx:74LS00
- added unit 2 of U18
- U1, U10, U11, U14, U17, U3, U8, U9: footprint Package_DIP:DIP-20_W7.62mm_Socket -> Package_SO:SO-20_12.8x7.5mm_P1.27mm
Connections:
- net +5V: now also U22.14 (VCC), U4.14 (VCC); no longer U22.7 (GND), U4.7 (GND)
- net GND: now also U22.7 (GND), U4.7 (GND); no longer U22.14 (VCC), U4.14 (VCC)
- net at J2.1 (Pin_1): now also U18.6
- net at J1.65 (Sup): now also U18.4, U18.5
Other:
- moved on the sheet: U19E, U22E, U4E

Commit message: Added gerber files to Activation Module and corrected PinHeader
Parts:
- J1: footprint Computer_Component_Library:PinSocket_1x78_P2.00mm_Horizontal -> Computer_Component_Library:PinHeader_1x78_P2.54mm_Horizontal
Changed lines of the file:
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@@
     (property "Reference" "J1" (id 0) (at 321.6148 17.145 0))
     (property "Value" "Bus_Connector" (id 1) (at 321.6148 19.4564 0))
-    (property "Footprint" "Computer_Component_Library:PinSocket_1x78_P2.00mm_Horizontal" (id 2) (at 292.1 41.91 0)
+    (property "Footprint" "Computer_Component_Library:PinHeader_1x78_P2.54mm_Horizontal" (id 2) (at 292.1 41.91 0)
       (effects (font (size 1.27 1.27)) hide)
     )
@@
       (effects (font (size 1.27 1.27)) (justify right))
     )
-    (property "Footprint" "Computer_Component_Library:PinSocket_1x78_P2.00mm_Horizontal" (id 2) (at 356.87 101.6 0)
+    (property "Footprint" "Computer_Component_Library:PinHeader_1x78_P2.54mm_Horizontal" (id 2) (at 356.87 101.6 0)
       (effects (font (size 1.27 1.27)) hide)
     )
@@
       (effects (font (size 1.27 1.27)) (justify right))
     )
-    (property "Footprint" "Computer_Component_Library:PinSocket_1x78_P2.00mm_Horizontal" (id 2) (at 137.16 303.53 0)
+    (property "Footprint" "Computer_Component_Library:PinHeader_1x78_P2.54mm_Horizontal" (id 2) (at 137.16 303.53 0)
       (effects (font (size 1.27 1.27)) hide)
     )
@@
       (effects (font (size 1.27 1.27)) (justify right))
     )
-    (property "Footprint" "Computer_Component_Library:PinSocket_1x78_P2.00mm_Horizontal" (id 2) (at 270.51 303.53 0)
+    (property "Footprint" "Computer_Component_Library:PinHeader_1x78_P2.54mm_Horizontal" (id 2) (at 270.51 303.53 0)
       (effects (font (size 1.27 1.27)) hide)
     )
@@
       (effects (font (size 1.27 1.27)) (justify left))
     )
-    (property "Footprint" "Computer_Component_Library:PinSocket_1x78_P2.00mm_Horizontal" (id 2) (at 27.94 -7.62 0)
+    (property "Footprint" "Computer_Component_Library:PinHeader_1x78_P2.54mm_Horizontal" (id 2) (at 27.94 -7.62 0)
       (effects (font (size 1.27 1.27)) hide)
     )
@@
       (effects (font (size 1.27 1.27)) (justify left))
     )
-    (property "Footprint" "Computer_Component_Library:PinSocket_1x78_P2.00mm_Horizontal" (id 2) (at 6.35 -7.62 0)
+    (property "Footprint" "Computer_Component_Library:PinHeader_1x78_P2.54mm_Horizontal" (id 2) (at 6.35 -7.62 0)
       (effects (font (size 1.27 1.27)) hide)
     )
@@
       (effects (font (size 1.27 1.27)) (justify left))
     )
-    (property "Footprint" "Computer_Component_Library:PinSocket_1x78_P2.00mm_Horizontal" (id 2) (at 170.18 -7.62 0)
+    (property "Footprint" "Computer_Component_Library:PinHeader_1x78_P2.54mm_Horizontal" (id 2) (at 170.18 -7.62 0)
       (effects (font (size 1.27 1.27)) hide)
     )
@@
       (effects (font (size 1.27 1.27)) (justify left))
     )
-    (property "Footprint" "Computer_Component_Library:PinSocket_1x78_P2.00mm_Horizontal" (id 2) (at 147.32 -7.62 0)
+    (property "Footprint" "Computer_Component_Library:PinHeader_1x78_P2.54mm_Horizontal" (id 2) (at 147.32 -7.62 0)
       (effects (font (size 1.27 1.27)) hide)
     )
@@
     )
     (path "/00000000-0000-0000-0000-00006c2eefff"
-      (reference "J1") (unit 1) (value "Bus_Connector") (footprint "Computer_Component_Library:PinSocket_1x78_P2.00mm_Horizontal")
+      (reference "J1") (unit 1) (value "Bus_Connector") (footprint "Computer_Component_Library:PinHeader_1x78_P2.54mm_Horizontal")
     )
     (path "/00000000-0000-0000-0000-00006c4cbfa6"
-      (reference "J1") (unit 2) (value "Bus_Connector") (footprint "Computer_Component_Library:PinSocket_1x78_P2.00mm_Horizontal")
+      (reference "J1") (unit 2) (value "Bus_Connector") (footprint "Computer_Component_Library:PinHeader_1x78_P2.54mm_Horizontal")
     )
     (path "/00000000-0000-0000-0000-00006c4dedf9"
-      (reference "J1") (unit 3) (value "Bus_Connector") (footprint "Computer_Component_Library:PinSocket_1x78_P2.00mm_Horizontal")
+      (reference "J1") (unit 3) (value "Bus_Connector") (footprint "Computer_Component_Library:PinHeader_1x78_P2.54mm_Horizontal")
     )
     (path "/00000000-0000-0000-0000-00006c4e28ea"
-      (reference "J1") (unit 4) (value "Bus_Connector") (footprint "Computer_Component_Library:PinSocket_1x78_P2.00mm_Horizontal")
+      (reference "J1") (unit 4) (value "Bus_Connector") (footprint "Computer_Component_Library:PinHeader_1x78_P2.54mm_Horizontal")
     )
     (path "/00000000-0000-0000-0000-00006c5048a1"
-      (reference "J1") (unit 5) (value "Bus_Connector") (footprint "Computer_Component_Library:PinSocket_1x78_P2.00mm_Horizontal")
+      (reference "J1") (unit 5) (value "Bus_Connector") (footprint "Computer_Component_Library:PinHeader_1x78_P2.54mm_Horizontal")
     )
     (path "/00000000-0000-0000-0000-00006c50bf66"
-      (reference "J1") (unit 6) (value "Bus_Connector") (footprint "Computer_Component_Library:PinSocket_1x78_P2.00mm_Horizontal")
+      (reference "J1") (unit 6) (value "Bus_Connector") (footprint "Computer_Component_Library:PinHeader_1x78_P2.54mm_Horizontal")
     )
     (path "/00000000-0000-0000-0000-00006c51e5d0"
-      (reference "J1") (unit 7) (value "Bus_Connector") (footprint "Computer_Component_Library:PinSocket_1x78_P2.00mm_Horizontal")
+      (reference "J1") (unit 7) (value "Bus_Connector") (footprint "Computer_Component_Library:PinHeader_1x78_P2.54mm_Horizontal")
     )
     (path "/00000000-0000-0000-0000-0000620c9ffe"
-      (reference "J1") (unit 10) (value "Bus_Connector") (footprint "Computer_Component_Library:PinSocket_1x78_P2.00mm_Horizontal")
+      (reference "J1") (unit 10) (value "Bus_Connector") (footprint "Computer_Component_Library:PinHeader_1x78_P2.54mm_Horizontal")
     )
     (path "/00000000-0000-0000-0000-0000620b82f3"
