File: circets/Memory/memory/memory.kicad_pcb (KiCad board)
At the start: 2 copper layers, 152 x 199.5 mm, 23 parts, among them J1 Bus_Connector, J2 Bank_Controller_Enable_Out, J3 A_Bank_Out, J4 D_Bank_IO, U1 74LS00, U10 AS6C62256-55PCN, U11 28C256, U12 AS6C62256-55PCN, U2 74LS00, U3 74LS139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

Commit message: Added Name to Module and Removed old schematic pdfs
Other:
- outline, holes or cut-outs redrawn
- board text added: "Memory Rev v0.3"
Changed lines of the file:
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@@
     (title "Memory")
     (date "2022-02-14")
-    (rev "v.1")
+    (rev "v.3")
     (comment 2 "https://github.com/jufo-ufo/Breadboard-Computer/blob/master/LICENSE")
     (comment 3 "License: Apache License 2.0")
@@
   )
   (gr_line (start 27.5 217.5) (end 23 217.5) (layer "Edge.Cuts") (width 0.2))
-  (gr_line (start 175 18) (end 175 147) (layer "Edge.Cuts") (width 0.2))
-  (gr_line (start 175 147) (end 27.5 147) (layer "Edge.Cuts") (width 0.2))
+  (gr_line (start 175 18) (end 175 163) (layer "Edge.Cuts") (width 0.2))
+  (gr_line (start 175 163) (end 27.5 163) (layer "Edge.Cuts") (width 0.2))
   (gr_line (start 23 18) (end 175 18) (layer "Edge.Cuts") (width 0.2))
-  (gr_line (start 27.5 147) (end 27.5 217.5) (layer "Edge.Cuts") (width 0.2))
+  (gr_line (start 27.5 163) (end 27.5 217.5) (layer "Edge.Cuts") (width 0.2))
   (gr_line (start 23 18) (end 23 217.5) (layer "Edge.Cuts") (width 0.2))
   (gr_text "RE_ROM\n" (at 115.2 30.8 90) (layer "F.SilkS")
@@
     (effects (font (size 1.5 1.5) (thickness 0.3)))
   )
+  (gr_text "Memory\nRev v0.3\n" (at 100 154) (layer "F.SilkS")
+    (effects (font (size 5 5) (thickness 0.5)))
+  )
   (dimension (type aligned) (layer "Dwgs.User")
